File: PCB/vmodvga.kicad_pcb (KiCad board)
At the start: 2 copper layers, 0 parts

Commit message: Initial component placement
Parts:
- added C10: 47nf, SM0805, F.Cu at (227.5, 86.5)
- added C11: 1nf, SM0805, F.Cu at (222.8, 86.3)
- added C12: 47nf, SM0805, F.Cu at (201.7, 147.3)
- added C13: 47nf, SM0805, F.Cu at (225.5, 80.8)
- added C14: 10uf, SM0805, F.Cu at (131.8, 129.5)
- added C15: 8.2nf, SM0805, F.Cu at (125.2, 147.9)
- added C16: 82nf, SM0805, F.Cu at (125.2, 150.2)
- added C17: .1uf, SM0805, F.Cu at (121.3, 164.6)
- added C18: .1uf, SM0805, F.Cu at (121.3, 162.2)
- added C19: .1uf, SM0805, F.Cu at (121.2, 159.9)
- added C2: .1uf, SM0805, F.Cu at (57.1, 72.8)
- added C21: .1uf, SM0805, F.Cu at (146.2, 52.6)
- added C22: .1uf, SM0805, F.Cu at (146.2, 55.3)
- added C23: .1uf, SM0805, F.Cu at (146.5, 58.5)
- added C24: .1uf, SM0805, F.Cu at (146.7, 61.2)
- added C25: .1uf, SM0805, F.Cu at (146.9, 64.4)
- added C3: .1uf, SM0805, F.Cu at (59.9, 72.7)
- added C4: .1uf, SM0805, F.Cu at (62.8, 72.8)
- added C5: .1uf, SM0805, F.Cu at (65.9, 72.9)
- added C6: 47nf, SM0805, F.Cu at (201.8, 150.1)
- added C7: 47nf, SM0805, F.Cu at (219.6, 80.5)
- added C8: 47nf, SM0805, F.Cu at (197.6, 154.2)
- added C9: 1nf, SM0805, F.Cu at (197.6, 152.1)
- added Cp1: 47uf, -PANASONIC_D, F.Cu at (50.5, 53.6)
- added Cp2: 22uf, -PANASONIC_E, F.Cu at (125.9, 192.8)
- added Cp3: 22uf, -PANASONIC_E, F.Cu at (121.5, 170.7)
- added Cp4: 4.7uf, -PANASONIC_C, F.Cu at (141.6, 25.5)
- added Cp5: 22uf, -PANASONIC_E, F.Cu at (61.1, 64.2)
- added Cp6: 22uf, -PANASONIC_E, F.Cu at (146.2, 45.8)
- added FB1: FILTER, SM0805, F.Cu at (222.4, 75.6)
- added FB2: FILTER, SM0805, F.Cu at (224.9, 75.9)
- added FB3: FILTER, SM0805, F.Cu at (227.5, 75.7)
- added FB4: FILTER, SM0805, F.Cu at (206.4, 152.9)
- added FB5: FILTER, SM0805, F.Cu at (206.4, 155.4)
- added FB6: FILTER, SM0805, F.Cu at (206.4, 157.7)
- added J1: DE-15, DE-15, F.Cu at (224.2, 61.9)
- added J2: DE-15, DE-15, F.Cu at (212.5, 153.1)
- added J3: VHDCI, VHDCI, F.Cu at (51.8, 121.9)
- added R1: 75, SM0805, F.Cu at (222.5, 80.7)
- added R10: 10K, SM0805, F.Cu at (58.3, 144.7)
- added R11: 1K, SM0805, F.Cu at (62.9, 143.3)
- added R12: 1K, SM0805, F.Cu at (62.9, 140.9)
- added R13: 76.8k, SM0805, F.Cu at (125.4, 177.2)
- added R14: 147k, SM0805, F.Cu at (121.4, 177.2)
- added R15: 2.2K, SM0805, F.Cu at (58.2, 137.1)
- added R16: 2.2K, SM0805, F.Cu at (58.2, 139.1)
- added R17: 76.8k, SM0805, F.Cu at (142.1, 39.2)
- added R18: 147k, SM0805, F.Cu at (145.7, 39.2)
- added R2: 75, SM0805, F.Cu at (202.0, 153.0)
- added R3: 75, SM0805, F.Cu at (225.3, 86.3)
- added R4: 75, SM0805, F.Cu at (197.6, 156.3)
- added R5: 75, SM0805, F.Cu at (227.7, 80.7)
- added R6: 75, SM0805, F.Cu at (202.1, 157.8)
- added R7: 1K, SM0805, F.Cu at (58.5, 148.1)
- added R8: 1.5K, SM0805, F.Cu at (128.8, 149.1)
- added R9: 10K, SM0805, F.Cu at (58.3, 142.5)
- added U1: ADP3303-3V3, -SOIC8, F.Cu at (52.4, 64.3)
- added U2: ADP3334, -SOIC8, F.Cu at (125.4, 183.4)
- added U3: AD9984, analog-devices2-LQFP80, F.Cu at (120.9, 135.1)
- added U4: ADP3334, -SOIC8, F.Cu at (141.6, 33.7)
