File: PCB/vgaExp.sch (KiCad schematic (older format))
At the start: 41 parts, among them J1 DE-15, J2 DE-15, J3 VHDCI, P5 CONN_1, P6 CONN_1, P7 CONN_6, U3 AD9984

Commit message: Routing complete. Also Fixes #6
Connections:
- net SCL_VGA_RX_BUF: now also J3.37 (IO2_N); no longer J3.35 (IO1_N)
- net SDA_VGA_RX_BUF: now also J3.35 (IO1_N); no longer J3.37 (IO2_N)
Changed lines of the file:
@@
 Sheet 1 3
 Title ""
-Date "21 jul 2014"
+Date "24 jul 2014"
 Rev ""
 Comp ""
@@
 NoConn ~ 1500 1400
 NoConn ~ 1500 3100
+Text Label 10700 1000 0    47   ~ 0
+SDA_VGA_RX_BUF
 Text Label 10700 1200 0    47   ~ 0
-SDA_VGA_RX_BUF
-Text Label 10700 1000 0    47   ~ 0
 SCL_VGA_RX_BUF
 Text Label 10700 4000 0    47   ~ 0
