File: PCB/vgaExp.kicad_pcb (KiCad board)
At the start: 2 copper layers, 80 x 91.1 mm, 83 parts, among them J1 DE-15, J2 DE-15, J3 VHDCI, P5 CONN_1, P6 CONN_1, P7 CONN_6, U1 ADP3303-3V3, U2 ADP3334, U3 AD9984, U4 ADP3334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

Commit message: Gerbers
Parts:
- -: value - -> (none)
- FB4, FB5, FB6: value FILTER -> (none)
- P5, P6: value CONN_1 -> (none)
- P7: value CONN_6 -> (none)
- R14: value R147K -> 147K
- TP1, TP10, TP11, TP12, TP13, TP2, TP3, TP4, TP5, TP6, TP7, TP8, TP9: value TESTPOINT -> (none)
Routing:
- net /HSOUT: track 57.2 -> 43.9 mm
- net /I2C/DDC Section/GND: track 150.9 -> 141.8 mm
- net (no net): track 0.00 -> 1.12 mm, vias 0 -> 1

Commit message: Rev: v02 without length-matching
Routing:
- net /I2C/DDC Section/GND: track 141.8 -> 143.2 mm
- net (no net): track 1.12 -> 0.00 mm, vias 1 -> 0
Other:
- board text added: "(C) Rohit - CC BY-SA 4.0 or TAPR 1.0"
Changed lines of the file:
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@@
     (area 54.348284 17.969177 168.150001 110.947)
     (thickness 1.6)
-    (drawings 65)
-    (tracks 1153)
+    (drawings 66)
+    (tracks 1152)
     (zones 0)
     (modules 83)
@@
   (page A3)
   (layers
-    (15 F.Cu signal hide)
-    (0 B.Cu signal hide)
+    (15 F.Cu signal)
+    (0 B.Cu signal)
     (16 B.Adhes user)
     (17 F.Adhes user)
@@
   )
   (setup
-    (last_trace_width 0.125)
+    (last_trace_width 0.5)
     (user_trace_width 0.13)
     (user_trace_width 0.2032)
@@
     (pad_to_mask_clearance 0)
     (aux_axis_origin 0 0)
-    (visible_elements 7FFFDFFF)
+    (visible_elements 7FFFFFFF)
     (pcbplotparams
       (layerselection 284196865)
@@
   (module DE-15 (layer F.Cu)
     (at 110.7 24.5 180)
-    (fp_text reference J2 (at -12.66 -5.7 180) (layer F.SilkS)
+    (fp_text reference J2 (at -10.5 -5.5 180) (layer F.SilkS)
       (effects (font (size 1 1) (thickness 0.15)))
     )
@@
   (module DE-15 (layer F.Cu)
     (at 145.8 24.5 180)
-    (fp_text reference J1 (at -12.66 -5.7 180) (layer F.SilkS)
+    (fp_text reference J1 (at -10 -4.8 180) (layer F.SilkS)
       (effects (font (size 1 1) (thickness 0.15)))
     )
@@
     (tags "SMALL OUTLINE IC")
     (attr smd)
-    (fp_text reference U5 (at 0.05 -0.14 180) (layer B.SilkS)
+    (fp_text reference U5 (at -0.25 -0.64 180) (layer B.SilkS) hide
       (effects (font (size 1.27 1.27) (thickness 0.0889)))
     )
-    (fp_text value 24AA014 (at 3.85 0.06 270) (layer B.SilkS)
+    (fp_text value 24AA014 (at 3.75 0.26 270) (layer B.SilkS) hide
       (effects (font (size 1.27 1.27) (thickness 0.0889)))
     )
@@
     )
   )
+  (gr_text "(C) Rohit - CC BY-SA 4.0 or TAPR 1.0" (at 129.3 106.6) (layer B.SilkS)
+    (effects (font (size 1.5 1.5) (thickness 0.3) italic) (justify mirror))
+  )
   (gr_text "V.Reg: OVDD" (at 149.35 87.39) (layer B.SilkS)
     (effects (font (size 1.5 1.5) (thickness 0.3)) (justify mirror))
@@
   (gr_line (start 87.9 18.2418) (end 167.9 18.2418) (angle 90) (layer Edge.Cuts) (width 0.5))
   (gr_line (start 167.9 109.35) (end 87.9 109.35) (angle 90) (layer Edge.Cuts) (width 0.5))
-  (via (at 138.0579 41.9679) (size 0.45) (layers F.Cu B.Cu) (net 0))
-  (segment (start 138.0579 41.9679) (end 138.06 41.97) (width 0.25) (layer B.Cu) (net 0))
-  (segment (start 138.0579 40.8525) (end 138.0579 41.9679) (width 0.25) (layer F.Cu) (net 0))
-  (segment (start 138.0579 41.9679) (end 138.06 41.97) (width 0.25) (layer F.Cu) (net 0))
   (segment (start 126.06 31.93) (end 129.16 31.93) (width 0.25) (layer B.Cu) (net 1))
   (segment (start 110.7 28.86) (end 113.77 31.93) (width 0.25) (layer B.Cu) (net 1))
@@
   (segment (start 112.39 22.56) (end 117.7 22.56) (width 0.25) (layer F.Cu) (net 27))
   (segment (start 110.7 24.25) (end 112.39 22.56) (width 0.25) (layer F.Cu) (net 27))
+  (segment (start 107.75 62.7225) (end 108.1225 62.7225) (width 0.5) (layer B.Cu) (net 28) (status C00000))
+  (segment (start 108.1225 62.7225) (end 108.5 63.1) (width 0.5) (layer B.Cu) (net 28) (status 400000))
+  (segment (start 108.1225 62.7225) (end 108.5 63.1) (width 0.5) (layer B.Cu) (net 28) (status 400000))
   (segment (start 108.83 64.1375) (end 108.1975 64.1375) (width 0.5) (layer B.Cu) (net 28))
   (segment (start 108.1975 64.1375) (end 107.71 63.65) (width 0.5) (layer B.Cu) (net 28))
