File: GSoC_Designs/powerSupply.sch (KiCad schematic (older format))
At the start: 25 parts, among them U1 ADP3303-3V3, U2 ADP3334, U4 ADP3334

Commit message: Fixed the feedback circuit for ADP3334 ICs in schematic
Fixed the feedback circuit for ADP3334 Variable o/p voltage LDO ICs
which was resulting in incorrect output voltages on PD and VD lines.
Connections:
- wire segments 44 -> 47
Other:
- moved on the sheet: R13, R17
Changed lines of the file:
@@
 Sheet 2 2
 Title ""
-Date "15 may 2014"
+Date "31 may 2014"
 Rev ""
 Comp ""
@@
 L R R13
 U 1 1 537281D1
-P 6000 2000
-F 0 "R13" V 6080 2000 40  0000 C CNN
-F 1 "R" V 6007 2001 40  0000 C CNN
-F 2 "~" V 5930 2000 30  0000 C CNN
-F 3 "~" H 6000 2000 30  0000 C CNN
-	1    6000 2000
-	0    -1   -1   0
+P 5950 2050
+F 0 "R13" V 6030 2050 40  0000 C CNN
+F 1 "R" V 5957 2051 40  0000 C CNN
+F 2 "~" V 5880 2050 30  0000 C CNN
+F 3 "~" H 5950 2050 30  0000 C CNN
+	1    5950 2050
+	0    1    1    0
 $EndComp
 $Comp
@@
 L R R17
 U 1 1 53728791
-P 8400 4150
-F 0 "R17" V 8480 4150 40  0000 C CNN
-F 1 "R" V 8407 4151 40  0000 C CNN
-F 2 "~" V 8330 4150 30  0000 C CNN
-F 3 "~" H 8400 4150 30  0000 C CNN
-	1    8400 4150
+P 8350 4200
+F 0 "R17" V 8430 4200 40  0000 C CNN
+F 1 "R" V 8357 4201 40  0000 C CNN
+F 2 "~" V 8280 4200 30  0000 C CNN
+F 3 "~" H 8350 4200 30  0000 C CNN
+	1    8350 4200
 	0    -1   -1   0
 $EndComp
@@
 Connection ~ 3150 4450
 Wire Wire Line
-	5600 1950 5700 1950
+	5600 1950 6500 1950
 Wire Wire Line
 	5700 1950 5700 2050
 Wire Wire Line
 	5700 2050 5600 2050
-Wire Wire Line
-	5700 2000 5750 2000
-Connection ~ 5700 2000
-Wire Wire Line
-	6250 2000 6250 2150
-Wire Wire Line
-	5600 2150 7450 2150
 Connection ~ 6250 2150
 Connection ~ 6500 2150
@@
 	8100 4100 8100 4200
 Wire Wire Line
-	8100 4100 8000 4100
-Wire Wire Line
-	8100 4150 8150 4150
-Connection ~ 8100 4150
-Wire Wire Line
-	8650 4150 8700 4150
-Wire Wire Line
-	8700 4150 8700 4300
-Wire Wire Line
-	8000 4300 10450 4300
+	8000 4100 8950 4100
+Wire Wire Line
+	8950 4300 10450 4300
 Connection ~ 8700 4300
 Connection ~ 8950 4300
@@
 Text HLabel 10450 4300 2    60   Output ~ 0
 VD
+Wire Wire Line
+	5600 2150 6250 2150
+Wire Wire Line
+	6250 2150 6250 2050
+Wire Wire Line
+	6250 2050 6200 2050
+Wire Wire Line
+	6500 2150 7450 2150
+Wire Wire Line
+	6500 1950 6500 2150
+Connection ~ 5700 1950
+Wire Wire Line
+	8700 4200 8700 4300
+Wire Wire Line
+	8700 4200 8600 4200
+Wire Wire Line
+	8700 4300 8000 4300
+Wire Wire Line
+	8950 4100 8950 4300
+Connection ~ 8100 4100
 $EndSCHEMATC

Commit message: Footprint assignment and PCB components placement
Parts assigned (along with updated VHDCI and QFP80 footprints) and
components placed just at same place as in previous design. Also, there
is one more project with longer pads for QFP80 footprint
Parts:
- C17, C18, C19, C2, C21, C22, C23, C24, C25, C3, C4, C5: value C -> 0.1uf
- Cp1: value CP1 -> 47uf
- Cp2, Cp3, Cp5, Cp6: value CP1 -> 22uf
- Cp4: value CP1 -> 4.7uf
- R13, R17: value R -> 76.8K
- R14: value R -> R147K
- R18: value R -> 147K
Changed lines of the file:
@@
 Sheet 2 2
 Title ""
-Date "31 may 2014"
+Date "2 jun 2014"
 Rev ""
 Comp ""
@@
 P 2800 4250
 F 0 "C2" H 2800 4350 40  0000 L CNN
-F 1 "C" H 2806 4165 40  0000 L CNN
+F 1 "0.1uf" H 2806 4165 40  0000 L CNN
 F 2 "~" H 2838 4100 30  0000 C CNN
 F 3 "~" H 2800 4250 60  0000 C CNN
@@
 P 1050 4950
 F 0 "Cp1" H 1100 5050 50  0000 L CNN
-F 1 "CP1" H 1100 4850 50  0000 L CNN
+F 1 "47uf" H 1100 4850 50  0000 L CNN
 F 2 "~" H 1050 4950 60  0000 C CNN
 F 3 "~" H 1050 4950 60  0000 C CNN
@@
 P 2450 4250
 F 0 "Cp5" H 2500 4350 50  0000 L CNN
-F 1 "CP1" H 2500 4150 50  0000 L CNN
+F 1 "22uf" H 2500 4150 50  0000 L CNN
 F 2 "~" H 2450 4250 60  0000 C CNN
 F 3 "~" H 2450 4250 60  0000 C CNN
@@
 P 3050 4250
 F 0 "C3" H 3050 4350 40  0000 L CNN
-F 1 "C" H 3056 4165 40  0000 L CNN
+F 1 "0.1uf" H 3056 4165 40  0000 L CNN
 F 2 "~" H 3088 4100 30  0000 C CNN
 F 3 "~" H 3050 4250 60  0000 C CNN
@@
 P 3250 4250
 F 0 "C4" H 3250 4350 40  0000 L CNN
-F 1 "C" H 3256 4165 40  0000 L CNN
+F 1 "0.1uf" H 3256 4165 40  0000 L CNN
 F 2 "~" H 3288 4100 30  0000 C CNN
 F 3 "~" H 3250 4250 60  0000 C CNN
@@
 P 3450 4250
 F 0 "C5" H 3450 4350 40  0000 L CNN
-F 1 "C" H 3456 4165 40  0000 L CNN
+F 1 "0.1uf" H 3456 4165 40  0000 L CNN
 F 2 "~" H 3488 4100 30  0000 C CNN
 F 3 "~" H 3450 4250 60  0000 C CNN
@@
 P 4500 2650
 F 0 "Cp2" H 4550 2750 50  0000 L CNN
-F 1 "CP1" H 4550 2550 50  0000 L CNN
+F 1 "22uf" H 4550 2550 50  0000 L CNN
 F 2 "~" H 4500 2650 60  0000 C CNN
 F 3 "~" H 4500 2650 60  0000 C CNN
@@
 P 6500 2350
 F 0 "Cp3" H 6550 2450 50  0000 L CNN
-F 1 "CP1" H 6550 2250 50  0000 L CNN
+F 1 "22uf" H 6550 2250 50  0000 L CNN
 F 2 "~" H 6500 2350 60  0000 C CNN
 F 3 "~" H 6500 2350 60  0000 C CNN
@@
 P 6750 2350
 F 0 "C17" H 6750 2450 40  0000 L CNN
-F 1 "C" H 6756 2265 40  0000 L CNN
+F 1 "0.1uf" H 6756 2265 40  0000 L CNN
 F 2 "~" H 6788 2200 30  0000 C CNN
 F 3 "~" H 6750 2350 60  0000 C CNN
@@
 P 6950 2350
 F 0 "C18" H 6950 2450 40  0000 L CNN
-F 1 "C" H 6956 2265 40  0000 L CNN
+F 1 "0.1uf" H 6956 2265 40  0000 L CNN
 F 2 "~" H 6988 2200 30  0000 C CNN
 F 3 "~" H 6950 2350 60  0000 C CNN
@@
 P 7150 2350
 F 0 "C19" H 7150 2450 40  0000 L CNN
-F 1 "C" H 7156 2265 40  0000 L CNN
+F 1 "0.1uf" H 7156 2265 40  0000 L CNN
 F 2 "~" H 7188 2200 30  0000 C CNN
 F 3 "~" H 7150 2350 60  0000 C CNN
@@
 P 5950 2050
 F 0 "R13" V 6030 2050 40  0000 C CNN
-F 1 "R" V 5957 2051 40  0000 C CNN
+F 1 "76.8K" V 5957 2051 40  0000 C CNN
 F 2 "~" V 5880 2050 30  0000 C CNN
 F 3 "~" H 5950 2050 30  0000 C CNN
 	1    5950 2050
-	0    1    1    0
+	0    -1   -1   0
 $EndComp
 $Comp
@@
 P 6250 2400
 F 0 "R14" V 6330 2400 40  0000 C CNN
-F 1 "R" V 6257 2401 40  0000 C CNN
+F 1 "R147K" V 6257 2401 40  0000 C CNN
 F 2 "~" V 6180 2400 30  0000 C CNN
 F 3 "~" H 6250 2400 30  0000 C CNN
@@
 P 6850 4750
 F 0 "Cp4" H 6900 4850 50  0000 L CNN
-F 1 "CP1" H 6900 4650 50  0000 L CNN
+F 1 "4.7uf" H 6900 4650 50  0000 L CNN
 F 2 "~" H 6850 4750 60  0000 C CNN
 F 3 "~" H 6850 4750 60  0000 C CNN
@@
 P 8350 4200
 F 0 "R17" V 8430 4200 40  0000 C CNN
-F 1 "R" V 8357 4201 40  0000 C CNN
+F 1 "76.8K" V 8357 4201 40  0000 C CNN
 F 2 "~" V 8280 4200 30  0000 C CNN
 F 3 "~" H 8350 4200 30  0000 C CNN
@@
 P 8700 4550
 F 0 "R18" V 8780 4550 40  0000 C CNN
-F 1 "R" V 8707 4551 40  0000 C CNN
+F 1 "147K" V 8707 4551 40  0000 C CNN
 F 2 "~" V 8630 4550 30  0000 C CNN
 F 3 "~" H 8700 4550 30  0000 C CNN
@@
 P 8950 4500
 F 0 "Cp6" H 9000 4600 50  0000 L CNN
-F 1 "CP1" H 9000 4400 50  0000 L CNN
+F 1 "22uf" H 9000 4400 50  0000 L CNN
 F 2 "~" H 8950 4500 60  0000 C CNN
 F 3 "~" H 8950 4500 60  0000 C CNN
@@
 P 9250 4500
 F 0 "C21" H 9250 4600 40  0000 L CNN
-F 1 "C" H 9256 4415 40  0000 L CNN
+F 1 "0.1uf" H 9256 4415 40  0000 L CNN
 F 2 "~" H 9288 4350 30  0000 C CNN
 F 3 "~" H 9250 4500 60  0000 C CNN
@@
 P 9450 4500
 F 0 "C22" H 9450 4600 40  0000 L CNN
-F 1 "C" H 9456 4415 40  0000 L CNN
+F 1 "0.1uf" H 9456 4415 40  0000 L CNN
 F 2 "~" H 9488 4350 30  0000 C CNN
 F 3 "~" H 9450 4500 60  0000 C CNN
@@
 P 9650 4500
 F 0 "C23" H 9650 4600 40  0000 L CNN
-F 1 "C" H 9656 4415 40  0000 L CNN
+F 1 "0.1uf" H 9656 4415 40  0000 L CNN
 F 2 "~" H 9688 4350 30  0000 C CNN
 F 3 "~" H 9650 4500 60  0000 C CNN
@@
 P 9850 4500
 F 0 "C24" H 9850 4600 40  0000 L CNN
-F 1 "C" H 9856 4415 40  0000 L CNN
+F 1 "0.1uf" H 9856 4415 40  0000 L CNN
 F 2 "~" H 9888 4350 30  0000 C CNN
 F 3 "~" H 9850 4500 60  0000 C CNN
@@
 P 10050 4500
 F 0 "C25" H 10050 4600 40  0000 L CNN
-F 1 "C" H 10056 4415 40  0000 L CNN
+F 1 "0.1uf" H 10056 4415 40  0000 L CNN
 F 2 "~" H 10088 4350 30  0000 C CNN
 F 3 "~" H 10050 4500 60  0000 C CNN
@@
 Wire Wire Line
 	8000 4100 8950 4100
-Wire Wire Line
-	8950 4300 10450 4300
 Connection ~ 8700 4300
 Connection ~ 8950 4300
@@
 VD
 Wire Wire Line
-	5600 2150 6250 2150
-Wire Wire Line
-	6250 2150 6250 2050
-Wire Wire Line
-	6250 2050 6200 2050
-Wire Wire Line
-	6500 2150 7450 2150
+	6200 2050 6250 2050
+Wire Wire Line
+	6250 2050 6250 2150
+Wire Wire Line
+	6250 2150 5600 2150
 Wire Wire Line
 	6500 1950 6500 2150
 Connection ~ 5700 1950
 Wire Wire Line
-	8700 4200 8700 4300
+	6500 2150 7450 2150
+Wire Wire Line
+	8700 4300 8700 4200
 Wire Wire Line
 	8700 4200 8600 4200
@@
 	8950 4100 8950 4300
 Connection ~ 8100 4100
+Wire Wire Line
+	8950 4300 10450 4300
 $EndSCHEMATC
