File: GSoC_Designs/powerSupply.sch (KiCad schematic (older format))
At the start: 25 parts, among them U1 ADP3303-3V3, U2 ADP3334, U4 ADP3334

Commit message: All ERC Errors fixed
Connections:
- no-connect marks 3 -> 4
Changed lines of the file:
@@
 	1    0    0    -1
 $EndComp
+Text Label 7450 5100 0    60   ~ 0
+GND
+Text Label 6700 4250 0    60   ~ 0
+VCC
+Text Label 10300 4300 0    60   ~ 0
+VD
+Text HLabel 6700 4250 0    60   Input ~ 0
+VCC
+Text HLabel 3650 4050 2    60   Output ~ 0
+OVDD
+Text HLabel 7450 2150 2    60   Output ~ 0
+PVD
+Text HLabel 10450 4300 2    60   Output ~ 0
+VD
+Text HLabel 1700 5350 2    47   Input ~ 0
+GND
+Text HLabel 3150 4650 2    47   Input ~ 0
+GND
+Text HLabel 5050 3050 2    47   Input ~ 0
+GND
+Text HLabel 7450 5150 2    47   Input ~ 0
+GND
 Wire Wire Line
 	1050 4750 1600 4750
@@
 	1050 5150 2450 5150
 Wire Wire Line
-	1700 4750 1700 5300
+	1700 4750 1700 5350
 Wire Wire Line
 	2450 5150 2450 4450
@@
 Connection ~ 3250 4450
 Wire Wire Line
-	3150 4550 3150 4450
+	3150 4450 3150 4650
 Connection ~ 3150 4450
 Wire Wire Line
@@
 	6500 2850 6500 2550
 Wire Wire Line
-	5050 2950 5050 2850
+	5050 2850 5050 3050
 Connection ~ 5050 2850
 Connection ~ 7150 2150
@@
 Connection ~ 7400 5000
 Wire Wire Line
-	7450 5100 7450 5000
+	7450 5000 7450 5150
 Connection ~ 7450 5000
-Text Label 7450 5100 0    60   ~ 0
-GND
 Wire Wire Line
 	6850 4250 6850 4550
@@
 Connection ~ 6850 4400
 Connection ~ 6850 4250
-Text Label 6700 4250 0    60   ~ 0
-VCC
 Connection ~ 10050 4300
-Text Label 10300 4300 0    60   ~ 0
-VD
-Text HLabel 6700 4250 0    60   Input ~ 0
-VCC
-Text HLabel 3650 4050 2    60   Output ~ 0
-OVDD
-Text HLabel 7450 2150 2    60   Output ~ 0
-PVD
-Text HLabel 10450 4300 2    60   Output ~ 0
-VD
 Wire Wire Line
 	6200 2050 6250 2050
@@
 Wire Wire Line
 	8950 4300 10450 4300
+NoConn ~ 8000 4400
 $EndSCHEMATC
