File: GSoC_Designs/vgaExp_v01.sch (KiCad schematic (older format))
At the start: 43 parts, among them J1 DE-15, J2 DE-15, J3 VHDCI, P1 DIL16, P2 DIL16, P3 DIL16, P4 DIL16, U3 AD9984

Commit message: Footprint assignment and PCB components placement
Parts assigned (along with updated VHDCI and QFP80 footprints) and
components placed just at same place as in previous design. Also, there
is one more project with longer pads for QFP80 footprint
Parts:
- added P5, P6: CONN_1, symbol CONN_1
- C10, C12, C13, C6, C7, C8: value C -> 47nf
- C11, C9: value C -> 1nf
- C14: value C -> 10nf
- C15: value C -> 8.2nf
- C16: value C -> 82nf
- P1, P2, P3, P4: value DIL16 -> 50R
- R1, R3, R5: value R -> 75R
- R10, R9: value R -> 10K
- R11, R12, R7: value R -> 1K
- R15, R16: value R -> 2.2K
- R19, R20, R21, R22: value R -> 50R
- R2, R4, R6: value R -> 75
- R8: value R -> 1.5K
Changed lines of the file:
@@
 Sheet 1 2
 Title ""
-Date "31 may 2014"
+Date "2 jun 2014"
 Rev ""
 Comp ""
@@
 U 1 1 537486B2
 P 7850 4350
-F 0 "P4" H 7850 4800 60  0000 C CNN
-F 1 "DIL16" V 7850 4350 50  0000 C CNN
+F 0 "P4" H 7850 3900 60  0000 C CNN
+F 1 "50R" V 7850 4350 50  0000 C CNN
 F 2 "" H 7850 4350 60  0000 C CNN
 F 3 "" H 7850 4350 60  0000 C CNN
@@
 U 1 1 537486BF
 P 5350 6000
-F 0 "P1" H 5350 6450 60  0000 C CNN
-F 1 "DIL16" V 5350 6000 50  0000 C CNN
+F 0 "P1" V 5350 6200 60  0000 C CNN
+F 1 "50R" V 5350 6000 50  0000 C CNN
 F 2 "" H 5350 6000 60  0000 C CNN
 F 3 "" H 5350 6000 60  0000 C CNN
@@
 U 1 1 537486C5
 P 7850 2950
-F 0 "P3" H 7850 3400 60  0000 C CNN
-F 1 "DIL16" V 7850 2950 50  0000 C CNN
+F 0 "P3" H 7850 2500 60  0000 C CNN
+F 1 "50R" V 7850 2950 50  0000 C CNN
 F 2 "" H 7850 2950 60  0000 C CNN
 F 3 "" H 7850 2950 60  0000 C CNN
@@
 U 1 1 537486CB
 P 6150 6000
-F 0 "P2" H 6150 6450 60  0000 C CNN
-F 1 "DIL16" V 6150 6000 50  0000 C CNN
+F 0 "P2" V 6150 6200 60  0000 C CNN
+F 1 "50R" V 6150 6000 50  0000 C CNN
 F 2 "" H 6150 6000 60  0000 C CNN
 F 3 "" H 6150 6000 60  0000 C CNN
@@
 U 1 1 53748A08
 P 7750 3400
-F 0 "R19" V 7830 3400 40  0000 C CNN
-F 1 "R" V 7757 3401 40  0000 C CNN
+F 0 "R19" V 7750 3300 40  0000 C CNN
+F 1 "50R" V 7750 3450 40  0000 C CNN
 F 2 "~" V 7680 3400 30  0000 C CNN
 F 3 "~" H 7750 3400 30  0000 C CNN
@@
 U 1 1 53748A39
 P 7750 3500
-F 0 "R20" V 7830 3500 40  0000 C CNN
-F 1 "R" V 7757 3501 40  0000 C CNN
+F 0 "R20" V 7750 3400 40  0000 C CNN
+F 1 "50R" V 7750 3550 40  0000 C CNN
 F 2 "~" V 7680 3500 30  0000 C CNN
 F 3 "~" H 7750 3500 30  0000 C CNN
@@
 U 1 1 53748A3F
 P 7750 3800
-F 0 "R21" V 7830 3800 40  0000 C CNN
-F 1 "R" V 7757 3801 40  0000 C CNN
+F 0 "R21" V 7750 3700 40  0000 C CNN
+F 1 "50R" V 7750 3850 40  0000 C CNN
 F 2 "~" V 7680 3800 30  0000 C CNN
 F 3 "~" H 7750 3800 30  0000 C CNN
@@
 U 1 1 53748A45
 P 7750 3900
-F 0 "R22" V 7830 3900 40  0000 C CNN
-F 1 "R" V 7757 3901 40  0000 C CNN
+F 0 "R22" V 7750 3800 40  0000 C CNN
+F 1 "50R" V 7750 3950 40  0000 C CNN
 F 2 "~" V 7680 3900 30  0000 C CNN
 F 3 "~" H 7750 3900 30  0000 C CNN
@@
 P 4350 6000
 F 0 "R9" V 4430 6000 40  0000 C CNN
-F 1 "R" V 4357 6001 40  0000 C CNN
+F 1 "10K" V 4357 6001 40  0000 C CNN
 F 2 "~" V 4280 6000 30  0000 C CNN
 F 3 "~" H 4350 6000 30  0000 C CNN
@@
 P 4350 6250
 F 0 "R10" V 4430 6250 40  0000 C CNN
-F 1 "R" V 4357 6251 40  0000 C CNN
+F 1 "10K" V 4357 6251 40  0000 C CNN
 F 2 "~" V 4280 6250 30  0000 C CNN
 F 3 "~" H 4350 6250 30  0000 C CNN
@@
 U 1 1 53748DA0
 P 6100 1950
-F 0 "R15" V 6180 1950 40  0000 C CNN
-F 1 "R" V 6107 1951 40  0000 C CNN
+F 0 "R15" V 6200 1850 40  0000 C CNN
+F 1 "2.2K" V 6107 1951 40  0000 C CNN
 F 2 "~" V 6030 1950 30  0000 C CNN
 F 3 "~" H 6100 1950 30  0000 C CNN
@@
 U 1 1 53748DA6
 P 6200 1950
-F 0 "R16" V 6280 1950 40  0000 C CNN
-F 1 "R" V 6207 1951 40  0000 C CNN
+F 0 "R16" V 6100 1850 40  0000 C CNN
+F 1 "2.2K" V 6207 1951 40  0000 C CNN
 F 2 "~" V 6130 1950 30  0000 C CNN
 F 3 "~" H 6200 1950 30  0000 C CNN
@@
 P 5200 1200
 F 0 "R11" V 5280 1200 40  0000 C CNN
-F 1 "R" V 5207 1201 40  0000 C CNN
+F 1 "1K" V 5207 1201 40  0000 C CNN
 F 2 "~" V 5130 1200 30  0000 C CNN
 F 3 "~" H 5200 1200 30  0000 C CNN
@@
 P 5200 1400
 F 0 "R12" V 5280 1400 40  0000 C CNN
-F 1 "R" V 5207 1401 40  0000 C CNN
+F 1 "1K" V 5207 1401 40  0000 C CNN
 F 2 "~" V 5130 1400 30  0000 C CNN
 F 3 "~" H 5200 1400 30  0000 C CNN
@@
 P 3800 1850
 F 0 "R8" V 3880 1850 40  0000 C CNN
-F 1 "R" V 3807 1851 40  0000 C CNN
+F 1 "1.5K" V 3807 1851 40  0000 C CNN
 F 2 "~" V 3730 1850 30  0000 C CNN
 F 3 "~" H 3800 1850 30  0000 C CNN
@@
 P 3450 2100
 F 0 "C16" H 3450 2200 40  0000 L CNN
-F 1 "C" H 3456 2015 40  0000 L CNN
+F 1 "82nf" H 3456 2015 40  0000 L CNN
 F 2 "~" H 3488 1950 30  0000 C CNN
 F 3 "~" H 3450 2100 60  0000 C CNN
@@
 P 3450 1600
 F 0 "C15" H 3450 1700 40  0000 L CNN
-F 1 "C" H 3456 1515 40  0000 L CNN
+F 1 "8.2nf" H 3456 1515 40  0000 L CNN
 F 2 "~" H 3488 1450 30  0000 C CNN
 F 3 "~" H 3450 1600 60  0000 C CNN
@@
 P 3500 3000
 F 0 "C6" H 3500 3100 40  0000 L CNN
-F 1 "C" H 3506 2915 40  0000 L CNN
+F 1 "47nf" H 3506 2915 40  0000 L CNN
 F 2 "~" H 3538 2850 30  0000 C CNN
 F 3 "~" H 3500 3000 60  0000 C CNN
@@
 P 3500 3200
 F 0 "C7" H 3500 3300 40  0000 L CNN
-F 1 "C" H 3506 3115 40  0000 L CNN
+F 1 "47nf" H 3506 3115 40  0000 L CNN
 F 2 "~" H 3538 3050 30  0000 C CNN
 F 3 "~" H 3500 3200 60  0000 C CNN
@@
 P 3500 3400
 F 0 "C8" H 3500 3500 40  0000 L CNN
-F 1 "C" H 3506 3315 40  0000 L CNN
+F 1 "47nf" H 3506 3315 40  0000 L CNN
 F 2 "~" H 3538 3250 30  0000 C CNN
 F 3 "~" H 3500 3400 60  0000 C CNN
@@
 P 3500 3600
 F 0 "C9" H 3500 3700 40  0000 L CNN
-F 1 "C" H 3506 3515 40  0000 L CNN
+F 1 "1nf" H 3506 3515 40  0000 L CNN
 F 2 "~" H 3538 3450 30  0000 C CNN
 F 3 "~" H 3500 3600 60  0000 C CNN
@@
 P 3500 3800
 F 0 "C10" H 3500 3900 40  0000 L CNN
-F 1 "C" H 3506 3715 40  0000 L CNN
+F 1 "47nf" H 3506 3715 40  0000 L CNN
 F 2 "~" H 3538 3650 30  0000 C CNN
 F 3 "~" H 3500 3800 60  0000 C CNN
@@
 P 3500 4000
 F 0 "C11" H 3500 4100 40  0000 L CNN
-F 1 "C" H 3506 3915 40  0000 L CNN
+F 1 "1nf" H 3506 3915 40  0000 L CNN
 F 2 "~" H 3538 3850 30  0000 C CNN
 F 3 "~" H 3500 4000 60  0000 C CNN
@@
 P 3500 4200
 F 0 "C12" H 3500 4300 40  0000 L CNN
-F 1 "C" H 3506 4115 40  0000 L CNN
+F 1 "47nf" H 3506 4115 40  0000 L CNN
 F 2 "~" H 3538 4050 30  0000 C CNN
 F 3 "~" H 3500 4200 60  0000 C CNN
@@
 P 3500 4400
 F 0 "C13" H 3500 4500 40  0000 L CNN
-F 1 "C" H 3506 4315 40  0000 L CNN
+F 1 "47nf" H 3506 4315 40  0000 L CNN
 F 2 "~" H 3538 4250 30  0000 C CNN
 F 3 "~" H 3500 4400 60  0000 C CNN
@@
 P 3700 4800
 F 0 "C14" H 3700 4900 40  0000 L CNN
-F 1 "C" H 3706 4715 40  0000 L CNN
+F 1 "10nf" H 3706 4715 40  0000 L CNN
 F 2 "~" H 3738 4650 30  0000 C CNN
 F 3 "~" H 3700 4800 60  0000 C CNN
@@
 P 2750 4700
 F 0 "R5" V 2830 4700 40  0000 C CNN
-F 1 "R" V 2757 4701 40  0000 C CNN
+F 1 "75R" V 2757 4701 40  0000 C CNN
 F 2 "~" V 2680 4700 30  0000 C CNN
 F 3 "~" H 2750 4700 30  0000 C CNN
@@
 P 2600 4700
 F 0 "R3" V 2680 4700 40  0000 C CNN
-F 1 "R" V 2607 4701 40  0000 C CNN
+F 1 "75R" V 2607 4701 40  0000 C CNN
 F 2 "~" V 2530 4700 30  0000 C CNN
 F 3 "~" H 2600 4700 30  0000 C CNN
@@
 P 2450 4700
 F 0 "R1" V 2530 4700 40  0000 C CNN
-F 1 "R" V 2457 4701 40  0000 C CNN
+F 1 "75R" V 2457 4701 40  0000 C CNN
 F 2 "~" V 2380 4700 30  0000 C CNN
 F 3 "~" H 2450 4700 30  0000 C CNN
@@
 P 2750 2150
 F 0 "R6" V 2830 2150 40  0000 C CNN
-F 1 "R" V 2757 2151 40  0000 C CNN
+F 1 "75" V 2757 2151 40  0000 C CNN
 F 2 "~" V 2680 2150 30  0000 C CNN
 F 3 "~" H 2750 2150 30  0000 C CNN
@@
 P 2600 2150
 F 0 "R4" V 2680 2150 40  0000 C CNN
-F 1 "R" V 2607 2151 40  0000 C CNN
+F 1 "75" V 2607 2151 40  0000 C CNN
 F 2 "~" V 2530 2150 30  0000 C CNN
 F 3 "~" H 2600 2150 30  0000 C CNN
@@
 P 2450 2150
 F 0 "R2" V 2530 2150 40  0000 C CNN
-F 1 "R" V 2457 2151 40  0000 C CNN
+F 1 "75" V 2457 2151 40  0000 C CNN
 F 2 "~" V 2380 2150 30  0000 C CNN
 F 3 "~" H 2450 2150 30  0000 C CNN
@@
 P 3250 4850
 F 0 "R7" V 3330 4850 40  0000 C CNN
-F 1 "R" V 3257 4851 40  0000 C CNN
+F 1 "1K" V 3257 4851 40  0000 C CNN
 F 2 "~" V 3180 4850 30  0000 C CNN
 F 3 "~" H 3250 4850 30  0000 C CNN
@@
 Text Label 10900 5750 0    60   ~ 0
 GND
+$Comp
+L CONN_1 P5
+U 1 1 538CC67A
+P 1150 5200
+F 0 "P5" H 1230 5200 40  0000 L CNN
+F 1 "CONN_1" H 1150 5255 30  0001 C CNN
+F 2 "" H 1150 5200 60  0000 C CNN
+F 3 "" H 1150 5200 60  0000 C CNN
+	1    1150 5200
+	1    0    0    -1
+$EndComp
+$Comp
+L CONN_1 P6
+U 1 1 538CC6E1
+P 1150 5300
+F 0 "P6" H 1230 5300 40  0000 L CNN
+F 1 "CONN_1" H 1150 5355 30  0001 C CNN
+F 2 "" H 1150 5300 60  0000 C CNN
+F 3 "" H 1150 5300 60  0000 C CNN
+	1    1150 5300
+	1    0    0    -1
+$EndComp
+Text Label 850  5200 0    60   ~ 0
+GND
+Text Label 850  5300 0    60   ~ 0
+VCC
 $EndSCHEMATC
