File: GSoC_Designs/vgaExp.sch (KiCad schematic (older format))
At the start: 45 parts, among them J1 DE-15, J2 DE-15, J3 VHDCI, P1 50R, P2 50R, P3 50R, P4 50R, P5 CONN_1, P6 CONN_1, U3 AD9984

Commit message: Fixed some ERC Errors
Connections:
- net labels added: PWD
- wire segments 205 -> 234
Changed lines of the file:
@@
 $EndComp
 $Sheet
-S 750  5800 1150 900
+S 2850 6650 1150 900
 U 53727A78
 F0 "PowerSupply" 50
 F1 "powerSupply.sch" 50
-F2 "VCC" I L 750 6000 60
-F3 "GND" I L 750 6650 60
-F4 "OVDD" O R 1900 6000 60
-F5 "PVD" O R 1900 6200 60
-F6 "VD" O R 1900 6400 60
-F7 "GND" O R 1900 6600 60
+F2 "VCC" I L 2850 6850 60
+F3 "GND" I L 2850 7500 60
+F4 "OVDD" O R 4000 6850 60
+F5 "PVD" O R 4000 7050 60
+F6 "VD" O R 4000 7250 60
+F7 "GND" O R 4000 7450 60
 $EndSheet
 $Comp
@@
 	0    -1   -1   0
 $EndComp
-Text Label 4800 2450 1    60   ~ 0
-GND
-Text Label 5100 2450 1    60   ~ 0
-GND
-Text Label 5300 2450 1    60   ~ 0
+Text Label 4800 2300 1    60   ~ 0
+GND
+Text Label 5100 2250 1    60   ~ 0
+GND
+Text Label 5300 2300 1    60   ~ 0
 GND
 Text Label 5200 1950 0    60   ~ 0
@@
 Text Label 9050 5250 2    60   ~ 0
 B0
-Text Label 9050 5450 2    60   ~ 0
+Text Label 9000 5500 2    60   ~ 0
 SDA
 Text Label 10500 2150 0    60   ~ 0
@@
 Text Label 10500 5250 0    60   ~ 0
 COST
-Text Label 10500 5450 0    60   ~ 0
+Text Label 10600 5550 0    60   ~ 0
 SCL
 Wire Wire Line
@@
 Connection ~ 3800 1600
 Wire Wire Line
-	4800 2350 4800 2500
-Wire Wire Line
-	5100 2350 5100 2500
-Wire Wire Line
-	5300 2350 5300 2500
+	4800 2300 4800 2500
+Wire Wire Line
+	5100 2250 5100 2500
+Wire Wire Line
+	5300 2300 5300 2500
 Wire Wire Line
 	4900 2050 4900 2500
@@
 	4650 6250 4600 6250
 Wire Wire Line
-	3950 6000 4100 6000
-Wire Wire Line
-	3950 6250 4100 6250
+	3900 6000 4100 6000
+Wire Wire Line
+	3900 6250 4100 6250
 Wire Wire Line
 	5000 6400 5000 6350
@@
 	2750 5050 2750 4950
 Wire Wire Line
-	2600 4950 2600 5150
+	2600 4950 2600 5200
 Connection ~ 2600 5050
 Wire Wire Line
@@
 	3250 4500 3250 4600
 Wire Wire Line
-	3250 5150 3250 5100
+	3250 5100 3250 5200
 Connection ~ 3250 4500
 Wire Wire Line
@@
 	10500 2250 10900 2250
 Wire Wire Line
-	10900 2250 10900 5700
+	10900 2250 10900 5750
 Wire Wire Line
 	10900 5350 10500 5350
@@
 VCC
 $Sheet
-S 2100 6450 1900 1250
+S 600  6400 1900 1250
 U 53BE83F2
 F0 "I2C/DDC Section" 50
 F1 "i2c.sch" 50
-F2 "SCL_VGA_RX" B L 2100 6900 60
-F3 "SDA_VGA_RX" B L 2100 7000 60
-F4 "SCL_VGA_TX" B L 2100 7250 60
-F5 "SDA_VGA_TX" B L 2100 7350 60
-F6 "SCL_INT" B R 4000 7350 60
-F7 "SDA_INT" B R 4000 7250 60
-F8 "SCL_VGA_RX_BUF" B R 4000 6650 60
-F9 "SDA_RX_VGA_BUF" B R 4000 6750 60
-F10 "SCL_TX_VGA_BUF" B R 4000 6950 60
-F11 "SDA_VGA_TX_BUF" B R 4000 7050 60
-F12 "VCC" I L 2100 6550 60
-F13 "OVDD" I L 2100 6650 60
-F14 "GND" I L 2100 7550 60
+F2 "SCL_VGA_RX" B L 600 6850 60
+F3 "SDA_VGA_RX" B L 600 6950 60
+F4 "SCL_VGA_TX" B L 600 7200 60
+F5 "SDA_VGA_TX" B L 600 7300 60
+F6 "SCL_INT" B R 2500 7300 60
+F7 "SDA_INT" B R 2500 7200 60
+F8 "SCL_VGA_RX_BUF" B R 2500 6600 60
+F9 "SDA_RX_VGA_BUF" B R 2500 6700 60
+F10 "SCL_TX_VGA_BUF" B R 2500 6900 60
+F11 "SDA_VGA_TX_BUF" B R 2500 7000 60
+F12 "VCC" I L 600 6500 60
+F13 "OVDD" I L 600 6600 60
+F14 "GND" I L 600 7500 60
 $EndSheet
+Wire Wire Line
+	3250 5200 3200 5200
+Wire Wire Line
+	5700 2350 5750 2350
+Wire Wire Line
+	5800 2350 5850 2350
+Wire Wire Line
+	5900 2350 5950 2350
+Wire Wire Line
+	6000 2350 6050 2350
+Wire Wire Line
+	6300 2350 6350 2350
+Wire Wire Line
+	6400 2350 6450 2350
+Wire Wire Line
+	850  5200 1000 5200
+Wire Wire Line
+	850  5300 1000 5300
+Wire Wire Line
+	2550 1700 2600 1700
+Wire Wire Line
+	7600 3600 7600 3650
+Wire Wire Line
+	7600 3700 7600 3750
+Wire Wire Line
+	6550 5450 6550 5200
+Wire Wire Line
+	6550 5200 6500 5200
+Wire Wire Line
+	6700 5200 6700 5400
+Wire Wire Line
+	5450 5350 5450 5200
+Wire Wire Line
+	5450 5200 5400 5200
+Wire Wire Line
+	5350 5350 5350 5200
+Wire Wire Line
+	5350 5200 5300 5200
+Wire Wire Line
+	9050 5450 9000 5450
+Wire Wire Line
+	9000 5450 9000 5500
+Wire Wire Line
+	10500 5450 10600 5450
+Wire Wire Line
+	10600 5450 10600 5550
+Wire Wire Line
+	2650 6850 2850 6850
+Text Label 2650 6850 0    60   ~ 0
+VCC
+Wire Wire Line
+	4000 6850 4200 6850
+Wire Wire Line
+	4000 7050 4200 7050
+Wire Wire Line
+	4000 7250 4200 7250
+Wire Wire Line
+	4000 7450 4200 7450
+Wire Wire Line
+	2700 7500 2850 7500
+Text Label 4200 6850 0    60   ~ 0
+OVDD
+Text Label 4200 7050 0    60   ~ 0
+PWD
+Text Label 4200 7250 0    60   ~ 0
+VD
+Text Label 4200 7450 0    60   ~ 0
+GND
+Text Label 2700 7500 2    60   ~ 0
+GND
 $EndSCHEMATC

Commit message: All ERC Errors fixed
Parts:
- removed FB1, FB2, FB3: FILTER, ~, symbol FILTER
- removed R1, R3, R5: 75R, ~, symbol R
Connections:
- net CLAMP: no longer J3.65 (IO18_N)
- net COST: no longer J3.66 (IO19_N)
- net GND: now also J1.10 (P10), J2.10 (P10); no longer J1.4 (P4), J1.9 (P9), J2.9 (P9)
- net HSYNC0: now also J1.13 (P13)
- net HSYNC1: no longer J1.13 (P13), U3.68 (HSYNC1)
- net OE_Field: no longer J3.35 (IO1_N)
- net PWRDWN: no longer J3.37 (IO2_N)
- net SCL: now also R15.1, U3.67 (SCL)
- net SDA: now also R16.1, U3.66 (SDA)
- net VSYNC0: now also J1.14 (P14)
- net VSYNC1: no longer J1.14 (P14), U3.69 (VSYNC1)
- net R: now reaches FB6.1, J2.1 (P1)
- net R: now also J1.1 (P1)
- net SDA_VGA_RX: now reaches J2.12 (P12)
- net SCL_VGA_RX: now reaches J2.15 (P15)
- net G: now reaches FB5.1, J2.2 (P2)
- net G: now also J1.2 (P2)
- net B: now reaches FB4.1, J2.3 (P3)
- net B: now also J1.3 (P3)
- net SDA_VGA_TX: now reaches J1.12 (P12)
- net SCL_VGA_TX: now reaches J1.15 (P15)
- net at C10.1: no longer C11.1
- new net SCL_VGA_RX_BUF: J3.65 (IO18_N)
- new net SCL_VGA_TX_BUF: J3.35 (IO1_N)
- new net SDA_VGA_RX_BUF: J3.66 (IO19_N)
- new net SDA_VGA_TX_BUF: J3.37 (IO2_N)
- no-connect marks 15 -> 19
Other:
- moved on the sheet: J3, P5, P6

Commit message: Added TestPoints
Parts:
- added TP1, TP10, TP11, TP12, TP13, TP2, TP3, TP4, TP5, TP6, TP7, TP8, TP9: TESTPOINT, symbol TESTPOINT
Connections:
- net DATACK: now also TP3.1
- net GND: now also TP13.1
- net HSOUT: now also TP5.1
- net HSYNC0: now also TP1.1
- net OVDD: now also TP9.1
- net SCL: now also TP7.1
- net SDA: now also TP8.1
- net SOGOUT: now also TP6.1
- net VCC: now also TP12.1
- net VD: now also TP10.1
- net VSOUT: now also TP4.1
- net VSYNC0: now also TP2.1
- new net PD: TP11.1
Other:
- note added: "Test Points"
