File: board/i2c.sch (KiCad schematic (older format))
At the start: 11 parts, among them U5 24AA014, U6 TCA9617A, U7 TCA9617A

Commit message: Upgrade schematic
Parts:
- R1, R23, R24, R25, R26, R27, R3, R5: symbol R -> R-RESCUE-vgaExp
Changed lines of the file:
@@
 EESchema Schematic File Version 2
+LIBS:vgaExp-rescue
 LIBS:power
 LIBS:device
@@
 LIBS:memory
 LIBS:xilinx
-LIBS:special
 LIBS:microcontrollers
 LIBS:dsp
@@
 LIBS:contrib
 LIBS:valves
-LIBS:24AA014
-LIBS:vmodvga
-LIBS:testpoint
 LIBS:vgaExp-cache
-EELAYER 27 0
+EELAYER 25 0
 EELAYER END
 $Descr A4 11693 8268
@@
 GND
 $Comp
-L R R5
+L R-RESCUE-vgaExp R5
 U 1 1 53C86281
 P 2650 2900
@@
 $EndComp
 $Comp
-L R R1
+L R-RESCUE-vgaExp R1
 U 1 1 53C8628E
 P 2450 2900
@@
 $EndComp
 $Comp
-L R R25
+L R-RESCUE-vgaExp R25
 U 1 1 53C86295
 P 5600 2850
@@
 $EndComp
 $Comp
-L R R26
+L R-RESCUE-vgaExp R26
 U 1 1 53C8629B
 P 5750 2850
@@
 $EndComp
 $Comp
-L R R3
+L R-RESCUE-vgaExp R3
 U 1 1 53C862A1
 P 2500 5000
@@
 $EndComp
 $Comp
-L R R23
+L R-RESCUE-vgaExp R23
 U 1 1 53C862A7
 P 2700 5000
@@
 $EndComp
 $Comp
-L R R24
+L R-RESCUE-vgaExp R24
 U 1 1 53C862AD
 P 5550 5050
@@
 $EndComp
 $Comp
-L R R27
+L R-RESCUE-vgaExp R27
 U 1 1 53C862B3
 P 5750 5050
