File: board/powerSupply.sch (KiCad schematic (older format))
At the start: 25 parts, among them U1 ADP3303-3V3, U2 ADP3334, U4 ADP3334

Commit message: Upgrade schematic
Parts:
- C17, C18, C19, C2, C21, C22, C23, C24, C25, C3, C4, C5: symbol C -> C-RESCUE-vgaExp
- Cp1, Cp2, Cp3, Cp4, Cp5, Cp6: symbol CP1 -> CP1-RESCUE-vgaExp
- R13, R14, R17, R18: symbol R -> R-RESCUE-vgaExp
- U1: symbol ADP3303-3V3 -> ADP3303-3v3
Changed lines of the file:
@@
 EESchema Schematic File Version 2
+LIBS:vgaExp-rescue
 LIBS:power
 LIBS:device
@@
 LIBS:memory
 LIBS:xilinx
-LIBS:special
 LIBS:microcontrollers
 LIBS:dsp
@@
 LIBS:contrib
 LIBS:valves
-LIBS:24AA014
-LIBS:vmodvga
-LIBS:testpoint
 LIBS:vgaExp-cache
-EELAYER 27 0
+EELAYER 25 0
 EELAYER END
 $Descr A4 11693 8268
@@
 $EndDescr
 $Comp
-L ADP3303-3V3 U1
+L ADP3303-3v3 U1
 U 1 1 53727ED8
 P 1700 4150
+AR Path="/53727ED8" Ref="U1"  Part="1"
+AR Path="/53727A78/53727ED8" Ref="U1"  Part="1"
 F 0 "U1" H 1800 3800 60  0000 C CNN
 F 1 "ADP3303-3V3" H 1750 4550 60  0000 C CNN
@@
 $EndComp
 $Comp
-L C C2
+L C-RESCUE-vgaExp C2
 U 1 1 53727F7A
 P 2800 4250
@@
 $EndComp
 $Comp
-L CP1 Cp1
+L CP1-RESCUE-vgaExp Cp1
 U 1 1 53727FAC
 P 1050 4950
@@
 $EndComp
 $Comp
-L CP1 Cp5
+L CP1-RESCUE-vgaExp Cp5
 U 1 1 53727FC3
 P 2450 4250
@@
 $EndComp
 $Comp
-L C C3
+L C-RESCUE-vgaExp C3
 U 1 1 53727FE7
 P 3050 4250
@@
 $EndComp
 $Comp
-L C C4
+L C-RESCUE-vgaExp C4
 U 1 1 53727FED
 P 3250 4250
@@
 $EndComp
 $Comp
-L C C5
+L C-RESCUE-vgaExp C5
 U 1 1 53727FF3
 P 3450 4250
@@
 NoConn ~ 2200 4200
 $Comp
-L CP1 Cp2
+L CP1-RESCUE-vgaExp Cp2
 U 1 1 537281B1
 P 4500 2650
@@
 $EndComp
 $Comp
-L CP1 Cp3
+L CP1-RESCUE-vgaExp Cp3
 U 1 1 537281B7
 P 6500 2350
@@
 $EndComp
 $Comp
-L C C17
+L C-RESCUE-vgaExp C17
 U 1 1 537281BD
 P 6750 2350
@@
 $EndComp
 $Comp
-L C C18
+L C-RESCUE-vgaExp C18
 U 1 1 537281C3
 P 6950 2350
@@
 $EndComp
 $Comp
-L C C19
+L C-RESCUE-vgaExp C19
 U 1 1 537281C9
 P 7150 2350
@@
 $EndComp
 $Comp
-L R R13
+L R-RESCUE-vgaExp R13
 U 1 1 537281D1
 P 5950 2050
@@
 $EndComp
 $Comp
-L R R14
+L R-RESCUE-vgaExp R14
 U 1 1 537281E8
 P 6250 2400
@@
 PVD
 $Comp
-L CP1 Cp4
+L CP1-RESCUE-vgaExp Cp4
 U 1 1 5372878B
 P 6850 4750
@@
 $EndComp
 $Comp
-L R R17
+L R-RESCUE-vgaExp R17
 U 1 1 53728791
 P 8350 4200
@@
 $EndComp
 $Comp
-L R R18
+L R-RESCUE-vgaExp R18
 U 1 1 53728797
 P 8700 4550
@@
 $EndComp
 $Comp
-L CP1 Cp6
+L CP1-RESCUE-vgaExp Cp6
 U 1 1 5372879D
 P 8950 4500
@@
 $EndComp
 $Comp
-L C C21
+L C-RESCUE-vgaExp C21
 U 1 1 537287A3
 P 9250 4500
@@
 $EndComp
 $Comp
-L C C22
+L C-RESCUE-vgaExp C22
 U 1 1 537287A9
 P 9450 4500
@@
 $EndComp
 $Comp
-L C C23
+L C-RESCUE-vgaExp C23
 U 1 1 537287AF
 P 9650 4500
@@
 $EndComp
 $Comp
-L C C24
+L C-RESCUE-vgaExp C24
 U 1 1 537287B5
 P 9850 4500
@@
 $EndComp
 $Comp
-L C C25
+L C-RESCUE-vgaExp C25
 U 1 1 537287BB
 P 10050 4500
