File: board/vgaExp.sch (KiCad schematic (older format))
At the start: 41 parts, among them J1 DE-15, J2 DE-15, J3 VHDCI, P5 CONN_1, P6 CONN_1, P7 CONN_6, U3 AD9984

Commit message: Upgrade schematic
Parts:
- C12, C14, C15, C16, C6, C8, C9: symbol C -> C-RESCUE-vgaExp
- R10, R11, R12, R15, R16, R2, R4, R6, R7, R8, R9: symbol R -> R-RESCUE-vgaExp
Changed lines of the file:
@@
 EESchema Schematic File Version 2
+LIBS:vgaExp-rescue
 LIBS:power
 LIBS:device
@@
 LIBS:memory
 LIBS:xilinx
-LIBS:special
 LIBS:microcontrollers
 LIBS:dsp
@@
 LIBS:contrib
 LIBS:valves
-LIBS:24AA014
-LIBS:vmodvga
-LIBS:testpoint
 LIBS:vgaExp-cache
-EELAYER 27 0
+EELAYER 25 0
 EELAYER END
 $Descr A4 11693 8268
@@
 $EndComp
 $Comp
-L R R9
+L R-RESCUE-vgaExp R9
 U 1 1 53748AFC
 P 4250 5200
@@
 $EndComp
 $Comp
-L R R10
+L R-RESCUE-vgaExp R10
 U 1 1 53748B02
 P 4250 5450
@@
 $EndComp
 $Comp
-L R R15
+L R-RESCUE-vgaExp R15
 U 1 1 53748DA0
 P 6100 1500
@@
 $EndComp
 $Comp
-L R R16
+L R-RESCUE-vgaExp R16
 U 1 1 53748DA6
 P 6200 1500
@@
 $EndComp
 $Comp
-L R R11
+L R-RESCUE-vgaExp R11
 U 1 1 53748DAC
 P 5200 750
@@
 $EndComp
 $Comp
-L R R12
+L R-RESCUE-vgaExp R12
 U 1 1 53748DD0
 P 5200 950
@@
 $EndComp
 $Comp
-L R R8
+L R-RESCUE-vgaExp R8
 U 1 1 53748DD6
 P 4350 1450
@@
 GND
 $Comp
-L C C16
+L C-RESCUE-vgaExp C16
 U 1 1 53749308
 P 3850 1450
@@
 $EndComp
 $Comp
-L C C15
+L C-RESCUE-vgaExp C15
 U 1 1 5374931F
 P 3850 1150
@@
 R0
 $Comp
-L C C6
+L C-RESCUE-vgaExp C6
 U 1 1 5374CA55
 P 3500 2550
@@
 $EndComp
 $Comp
-L C C8
+L C-RESCUE-vgaExp C8
 U 1 1 5374CAC1
 P 3500 2950
@@
 $EndComp
 $Comp
-L C C9
+L C-RESCUE-vgaExp C9
 U 1 1 5374CAC7
 P 3500 3150
@@
 $EndComp
 $Comp
-L C C12
+L C-RESCUE-vgaExp C12
 U 1 1 5374CAFD
 P 3500 3750
@@
 $EndComp
 $Comp
-L C C14
+L C-RESCUE-vgaExp C14
 U 1 1 5374CB09
 P 3700 4350
@@
 $EndComp
 $Comp
-L R R6
+L R-RESCUE-vgaExp R6
 U 1 1 5374CB7B
 P 2750 1700
@@
 $EndComp
 $Comp
-L R R4
+L R-RESCUE-vgaExp R4
 U 1 1 5374CB81
 P 2600 1700
@@
 $EndComp
 $Comp
-L R R2
+L R-RESCUE-vgaExp R2
 U 1 1 5374CB87
 P 2450 1700
@@
 $EndComp
 $Comp
-L R R7
+L R-RESCUE-vgaExp R7
 U 1 1 5374CB8D
 P 3250 4400
