File: board/vga.sch (KiCad schematic (older format))
At the start: 16 parts, among them P501 VGA RX I2C 3v, P502 VGA TX I2C 3v, P503 VGA RX I2C 5v, P504 VGA TX I2C 5v, P505 DE-15, P506 DE-15, U501 TCA9617A, U502 TCA9617A

Commit message: Start assigning footprints
Parts:
- P505, P506: footprint ~ -> (none)
- R501, R502, R503, R504, R505, R506, R507, R508: footprint (none) -> Resistors_SMD:R_0805_HandSoldering
Changed lines of the file:
@@
 F 0 "U502" H 5750 4950 60  0000 C CNN
 F 1 "TCA9617A" H 5750 5050 60  0000 C CNN
-F 2 "" H 6000 5100 60  0000 C CNN
+F 2 "" H 6000 5100 60  0001 C CNN
 F 3 "" H 6000 5100 60  0000 C CNN
 	1    5750 5000
@@
 F 0 "P506" V 8770 5600 60  0000 C CNN
 F 1 "DE-15" V 8880 5600 60  0000 C CNN
-F 2 "~" H 8800 5600 60  0000 C CNN
+F 2 "" H 8800 5600 60  0001 C CNN
 F 3 "~" H 8800 5600 60  0000 C CNN
 	1    8800 5600
@@
 VGA_R
 $Comp
-L GND #PWR510
+L GND #PWR041
 U 1 1 563F8497
 P 8200 5650
-F 0 "#PWR510" H 8200 5400 50  0001 C CNN
+F 0 "#PWR041" H 8200 5400 50  0001 C CNN
 F 1 "GND" H 8200 5500 50  0000 C CNN
 F 2 "" H 8200 5650 60  0000 C CNN
@@
 $EndComp
 $Comp
-L GND #PWR504
+L GND #PWR042
 U 1 1 563F85E4
 P 4300 5200
-F 0 "#PWR504" H 4300 4950 50  0001 C CNN
+F 0 "#PWR042" H 4300 4950 50  0001 C CNN
 F 1 "GND" V 4300 5000 50  0000 C CNN
 F 2 "" H 4300 5200 60  0000 C CNN
@@
 F 0 "R508" V 7730 4650 50  0000 C CNN
 F 1 "4K7" V 7650 4650 50  0000 C CNN
-F 2 "" V 7580 4650 30  0000 C CNN
+F 2 "Resistors_SMD:R_0805_HandSoldering" V 7580 4650 30  0001 C CNN
 F 3 "" H 7650 4650 30  0000 C CNN
 	1    7650 4650
@@
 F 0 "R506" V 7530 4650 50  0000 C CNN
 F 1 "4K7" V 7450 4650 50  0000 C CNN
-F 2 "" V 7380 4650 30  0000 C CNN
+F 2 "Resistors_SMD:R_0805_HandSoldering" V 7380 4650 30  0001 C CNN
 F 3 "" H 7450 4650 30  0000 C CNN
 	1    7450 4650
@@
 F 0 "R504" V 4280 4650 50  0000 C CNN
 F 1 "2K2" V 4200 4650 50  0000 C CNN
-F 2 "" V 4130 4650 30  0000 C CNN
+F 2 "Resistors_SMD:R_0805_HandSoldering" V 4130 4650 30  0001 C CNN
 F 3 "" H 4200 4650 30  0000 C CNN
 	1    4200 4650
@@
 F 0 "R502" V 4080 4650 50  0000 C CNN
 F 1 "2K2" V 4000 4650 50  0000 C CNN
-F 2 "" V 3930 4650 30  0000 C CNN
+F 2 "Resistors_SMD:R_0805_HandSoldering" V 3930 4650 30  0001 C CNN
 F 3 "" H 4000 4650 30  0000 C CNN
 	1    4000 4650
@@
 F 0 "U501" H 5750 1850 60  0000 C CNN
 F 1 "TCA9617A" H 5750 1950 60  0000 C CNN
-F 2 "" H 6000 2000 60  0000 C CNN
+F 2 "" H 6000 2000 60  0001 C CNN
 F 3 "" H 6000 2000 60  0000 C CNN
 	1    5750 1900
@@
 F 0 "P505" V 8770 2500 60  0000 C CNN
 F 1 "DE-15" V 8880 2500 60  0000 C CNN
-F 2 "~" H 8800 2500 60  0000 C CNN
+F 2 "" H 8800 2500 60  0001 C CNN
 F 3 "~" H 8800 2500 60  0000 C CNN
 	1    8800 2500
@@
 VGA_R
 $Comp
-L GND #PWR509
+L GND #PWR043
 U 1 1 5641B8E6
 P 8200 2550
-F 0 "#PWR509" H 8200 2300 50  0001 C CNN
+F 0 "#PWR043" H 8200 2300 50  0001 C CNN
 F 1 "GND" H 8200 2400 50  0000 C CNN
 F 2 "" H 8200 2550 60  0000 C CNN
@@
 $EndComp
 $Comp
-L GND #PWR502
+L GND #PWR044
 U 1 1 5641B8EC
 P 4300 2100
-F 0 "#PWR502" H 4300 1850 50  0001 C CNN
+F 0 "#PWR044" H 4300 1850 50  0001 C CNN
 F 1 "GND" V 4300 1900 50  0000 C CNN
 F 2 "" H 4300 2100 60  0000 C CNN
@@
 F 0 "R507" V 7730 1550 50  0000 C CNN
 F 1 "4K7" V 7650 1550 50  0000 C CNN
-F 2 "" V 7580 1550 30  0000 C CNN
+F 2 "Resistors_SMD:R_0805_HandSoldering" V 7580 1550 30  0001 C CNN
 F 3 "" H 7650 1550 30  0000 C CNN
 	1    7650 1550
@@
 F 0 "R505" V 7530 1550 50  0000 C CNN
 F 1 "4K7" V 7450 1550 50  0000 C CNN
-F 2 "" V 7380 1550 30  0000 C CNN
+F 2 "Resistors_SMD:R_0805_HandSoldering" V 7380 1550 30  0001 C CNN
 F 3 "" H 7450 1550 30  0000 C CNN
 	1    7450 1550
@@
 F 0 "R503" V 4280 1550 50  0000 C CNN
 F 1 "2K2" V 4200 1550 50  0000 C CNN
-F 2 "" V 4130 1550 30  0000 C CNN
+F 2 "Resistors_SMD:R_0805_HandSoldering" V 4130 1550 30  0001 C CNN
 F 3 "" H 4200 1550 30  0000 C CNN
 	1    4200 1550
@@
 F 0 "R501" V 4080 1550 50  0000 C CNN
 F 1 "2K2" V 4000 1550 50  0000 C CNN
-F 2 "" V 3930 1550 30  0000 C CNN
+F 2 "Resistors_SMD:R_0805_HandSoldering" V 3930 1550 30  0001 C CNN
 F 3 "" H 4000 1550 30  0000 C CNN
 	1    4000 1550
@@
 Connection ~ 7350 1300
 $Comp
-L +3V3 #PWR503
+L +3V3 #PWR045
 U 1 1 5641A682
 P 4300 4300
-F 0 "#PWR503" H 4300 4150 50  0001 C CNN
+F 0 "#PWR045" H 4300 4150 50  0001 C CNN
 F 1 "+3V3" H 4300 4440 50  0000 C CNN
 F 2 "" H 4300 4300 60  0000 C CNN
@@
 $EndComp
 $Comp
-L +3V3 #PWR501
+L +3V3 #PWR046
 U 1 1 5641A73F
 P 4300 1200
-F 0 "#PWR501" H 4300 1050 50  0001 C CNN
+F 0 "#PWR046" H 4300 1050 50  0001 C CNN
 F 1 "+3V3" H 4300 1340 50  0000 C CNN
 F 2 "" H 4300 1200 60  0000 C CNN
@@
 $EndComp
 $Comp
-L +5V #PWR507
+L +5V #PWR047
 U 1 1 56424FD7
 P 7350 1200
-F 0 "#PWR507" H 7350 1050 50  0001 C CNN
+F 0 "#PWR047" H 7350 1050 50  0001 C CNN
 F 1 "+5V" H 7350 1340 50  0000 C CNN
 F 2 "" H 7350 1200 60  0000 C CNN
@@
 $EndComp
 $Comp
-L +5V #PWR508
+L +5V #PWR048
 U 1 1 56425070
 P 7350 4300
-F 0 "#PWR508" H 7350 4150 50  0001 C CNN
+F 0 "#PWR048" H 7350 4150 50  0001 C CNN
 F 1 "+5V" H 7350 4440 50  0000 C CNN
 F 2 "" H 7350 4300 60  0000 C CNN
@@
 F 0 "P501" V 4650 2700 50  0000 C CNN
 F 1 "VGA RX I2C 3v" V 4750 2350 50  0000 C CNN
-F 2 "" H 4650 2350 50  0000 C CNN
+F 2 "" H 4650 2350 50  0001 C CNN
 F 3 "" H 4650 2350 50  0000 C CNN
 	1    4650 2350
@@
 F 0 "P502" V 4650 5800 50  0000 C CNN
 F 1 "VGA TX I2C 3v" V 4750 5450 50  0000 C CNN
-F 2 "" H 4650 5450 50  0000 C CNN
+F 2 "" H 4650 5450 50  0001 C CNN
 F 3 "" H 4650 5450 50  0000 C CNN
 	1    4650 5450
@@
 F 0 "P503" V 7000 2700 50  0000 C CNN
 F 1 "VGA RX I2C 5v" V 7100 2350 50  0000 C CNN
-F 2 "" H 7000 2350 50  0000 C CNN
+F 2 "" H 7000 2350 50  0001 C CNN
 F 3 "" H 7000 2350 50  0000 C CNN
 	1    7000 2350
@@
 $EndComp
 $Comp
-L GND #PWR505
+L GND #PWR049
 U 1 1 5692C822
 P 6850 2100
-F 0 "#PWR505" H 6850 1850 50  0001 C CNN
+F 0 "#PWR049" H 6850 1850 50  0001 C CNN
 F 1 "GND" H 6950 2100 50  0000 C CNN
 F 2 "" H 6850 2100 50  0000 C CNN
@@
 F 0 "P504" V 7000 5800 50  0000 C CNN
 F 1 "VGA TX I2C 5v" V 7100 5450 50  0000 C CNN
-F 2 "" H 7000 5450 50  0000 C CNN
+F 2 "" H 7000 5450 50  0001 C CNN
 F 3 "" H 7000 5450 50  0000 C CNN
 	1    7000 5450
@@
 $EndComp
 $Comp
-L GND #PWR506
+L GND #PWR050
 U 1 1 5692D0C6
 P 6850 5200
-F 0 "#PWR506" H 6850 4950 50  0001 C CNN
+F 0 "#PWR050" H 6850 4950 50  0001 C CNN
 F 1 "GND" H 6950 5200 50  0000 C CNN
 F 2 "" H 6850 5200 50  0000 C CNN

Commit message: More footprint assigning
Parts:
- P501, P502, P503, P504: footprint (none) -> CON-4X1-2.54:CON-2X1-2.54
Changed lines of the file:
@@
 F 0 "P501" V 4650 2700 50  0000 C CNN
 F 1 "VGA RX I2C 3v" V 4750 2350 50  0000 C CNN
-F 2 "" H 4650 2350 50  0001 C CNN
+F 2 "CON-4X1-2.54:CON-2X1-2.54" H 4650 2350 50  0001 C CNN
 F 3 "" H 4650 2350 50  0000 C CNN
 	1    4650 2350
@@
 F 0 "P502" V 4650 5800 50  0000 C CNN
 F 1 "VGA TX I2C 3v" V 4750 5450 50  0000 C CNN
-F 2 "" H 4650 5450 50  0001 C CNN
+F 2 "CON-4X1-2.54:CON-2X1-2.54" H 4650 5450 50  0001 C CNN
 F 3 "" H 4650 5450 50  0000 C CNN
 	1    4650 5450
@@
 F 0 "P503" V 7000 2700 50  0000 C CNN
 F 1 "VGA RX I2C 5v" V 7100 2350 50  0000 C CNN
-F 2 "" H 7000 2350 50  0001 C CNN
+F 2 "CON-4X1-2.54:CON-2X1-2.54" H 7000 2350 50  0001 C CNN
 F 3 "" H 7000 2350 50  0000 C CNN
 	1    7000 2350
@@
 F 0 "P504" V 7000 5800 50  0000 C CNN
 F 1 "VGA TX I2C 5v" V 7100 5450 50  0000 C CNN
-F 2 "" H 7000 5450 50  0001 C CNN
+F 2 "CON-4X1-2.54:CON-2X1-2.54" H 7000 5450 50  0001 C CNN
 F 3 "" H 7000 5450 50  0000 C CNN
 	1    7000 5450

Commit message: More footprints
Parts:
- P501, P502, P503, P504: footprint CON-4X1-2.54:CON-2X1-2.54 -> CON-SMD-2.54:CON-4X1-2.54
- P505, P506: footprint (none) -> DE-15:TE-1-1734530-1
- U501, U502: footprint (none) -> Housings_SSOP:MSOP-8_3x3mm_Pitch0.65mm
Changed lines of the file:
@@
 LIBS:testpoint
 LIBS:ad9984-power
+LIBS:3-rca
 EELAYER 25 0
 EELAYER END
@@
 F 0 "U502" H 5750 4950 60  0000 C CNN
 F 1 "TCA9617A" H 5750 5050 60  0000 C CNN
-F 2 "" H 6000 5100 60  0001 C CNN
+F 2 "Housings_SSOP:MSOP-8_3x3mm_Pitch0.65mm" H 6000 5100 60  0001 C CNN
 F 3 "" H 6000 5100 60  0000 C CNN
 	1    5750 5000
@@
 F 0 "P506" V 8770 5600 60  0000 C CNN
 F 1 "DE-15" V 8880 5600 60  0000 C CNN
-F 2 "" H 8800 5600 60  0001 C CNN
+F 2 "DE-15:TE-1-1734530-1" H 8800 5600 60  0001 C CNN
 F 3 "~" H 8800 5600 60  0000 C CNN
 	1    8800 5600
@@
 F 0 "U501" H 5750 1850 60  0000 C CNN
 F 1 "TCA9617A" H 5750 1950 60  0000 C CNN
-F 2 "" H 6000 2000 60  0001 C CNN
+F 2 "Housings_SSOP:MSOP-8_3x3mm_Pitch0.65mm" H 6000 2000 60  0001 C CNN
 F 3 "" H 6000 2000 60  0000 C CNN
 	1    5750 1900
@@
 F 0 "P505" V 8770 2500 60  0000 C CNN
 F 1 "DE-15" V 8880 2500 60  0000 C CNN
-F 2 "" H 8800 2500 60  0001 C CNN
+F 2 "DE-15:TE-1-1734530-1" H 8800 2500 60  0001 C CNN
 F 3 "~" H 8800 2500 60  0000 C CNN
 	1    8800 2500
@@
 F 0 "P501" V 4650 2700 50  0000 C CNN
 F 1 "VGA RX I2C 3v" V 4750 2350 50  0000 C CNN
-F 2 "CON-4X1-2.54:CON-2X1-2.54" H 4650 2350 50  0001 C CNN
+F 2 "CON-SMD-2.54:CON-4X1-2.54" H 4650 2350 50  0001 C CNN
 F 3 "" H 4650 2350 50  0000 C CNN
 	1    4650 2350
@@
 F 0 "P502" V 4650 5800 50  0000 C CNN
 F 1 "VGA TX I2C 3v" V 4750 5450 50  0000 C CNN
-F 2 "CON-4X1-2.54:CON-2X1-2.54" H 4650 5450 50  0001 C CNN
+F 2 "CON-SMD-2.54:CON-4X1-2.54" H 4650 5450 50  0001 C CNN
 F 3 "" H 4650 5450 50  0000 C CNN
 	1    4650 5450
@@
 F 0 "P503" V 7000 2700 50  0000 C CNN
 F 1 "VGA RX I2C 5v" V 7100 2350 50  0000 C CNN
-F 2 "CON-4X1-2.54:CON-2X1-2.54" H 7000 2350 50  0001 C CNN
+F 2 "CON-SMD-2.54:CON-4X1-2.54" H 7000 2350 50  0001 C CNN
 F 3 "" H 7000 2350 50  0000 C CNN
 	1    7000 2350
@@
 F 0 "P504" V 7000 5800 50  0000 C CNN
 F 1 "VGA TX I2C 5v" V 7100 5450 50  0000 C CNN
-F 2 "CON-4X1-2.54:CON-2X1-2.54" H 7000 5450 50  0001 C CNN
+F 2 "CON-SMD-2.54:CON-4X1-2.54" H 7000 5450 50  0001 C CNN
 F 3 "" H 7000 5450 50  0000 C CNN
 	1    7000 5450

Commit message: Finish footprint assignment
Parts:
- P501, P502, P503, P504: footprint CON-SMD-2.54:CON-4X1-2.54 -> CON-SMD-2.54:HARWIN-M20-87-4x1
Changed lines of the file:
@@
 F 0 "P501" V 4650 2700 50  0000 C CNN
 F 1 "VGA RX I2C 3v" V 4750 2350 50  0000 C CNN
-F 2 "CON-SMD-2.54:CON-4X1-2.54" H 4650 2350 50  0001 C CNN
+F 2 "CON-SMD-2.54:HARWIN-M20-87-4x1" H 4650 2350 50  0001 C CNN
 F 3 "" H 4650 2350 50  0000 C CNN
 	1    4650 2350
@@
 F 0 "P502" V 4650 5800 50  0000 C CNN
 F 1 "VGA TX I2C 3v" V 4750 5450 50  0000 C CNN
-F 2 "CON-SMD-2.54:CON-4X1-2.54" H 4650 5450 50  0001 C CNN
+F 2 "CON-SMD-2.54:HARWIN-M20-87-4x1" H 4650 5450 50  0001 C CNN
 F 3 "" H 4650 5450 50  0000 C CNN
 	1    4650 5450
@@
 F 0 "P503" V 7000 2700 50  0000 C CNN
 F 1 "VGA RX I2C 5v" V 7100 2350 50  0000 C CNN
-F 2 "CON-SMD-2.54:CON-4X1-2.54" H 7000 2350 50  0001 C CNN
+F 2 "CON-SMD-2.54:HARWIN-M20-87-4x1" H 7000 2350 50  0001 C CNN
 F 3 "" H 7000 2350 50  0000 C CNN
 	1    7000 2350
@@
 F 0 "P504" V 7000 5800 50  0000 C CNN
 F 1 "VGA TX I2C 5v" V 7100 5450 50  0000 C CNN
-F 2 "CON-SMD-2.54:CON-4X1-2.54" H 7000 5450 50  0001 C CNN
+F 2 "CON-SMD-2.54:HARWIN-M20-87-4x1" H 7000 5450 50  0001 C CNN
 F 3 "" H 7000 5450 50  0000 C CNN
 	1    7000 5450
