File: board/vga.sch (KiCad schematic (older format))
At the start: 36 parts, among them P601 3-RCA

Commit message: Assigning footprints.
Parts:
- CVI60, CVI61, CVI62, CVI63, CVI64, CVO60, CVO61, CVO62, CVO63, CVO64: footprint (none) -> Capacitors_SMD:C_1206_HandSoldering
- JVI60, JVO60: footprint (none) -> CON-SMD-2.54:HARWIN-M20-87-2x1
Changed lines of the file:
@@
 $EndComp
 $Comp
-L +3V3 #PWR048
+L +3V3 #PWR046
 U 1 1 5641A682
 P 5450 4100
-F 0 "#PWR048" H 5450 3950 50  0001 C CNN
+F 0 "#PWR046" H 5450 3950 50  0001 C CNN
 F 1 "+3V3" H 5450 4240 50  0000 C CNN
 F 2 "" H 5450 4100 60  0000 C CNN
@@
 COMP_Pr
 $Comp
-L GNDA #PWR054
+L GNDA #PWR047
 U 1 1 579715ED
 P 1850 4600
-F 0 "#PWR054" H 1850 4350 50  0001 C CNN
+F 0 "#PWR047" H 1850 4350 50  0001 C CNN
 F 1 "GNDA" H 1850 4450 50  0000 C CNN
 F 2 "" H 1850 4600 60  0000 C CNN
@@
 Analog VGA Signals\nNoise Sensitive
 $Comp
-L GNDA #PWR057
+L GNDA #PWR048
 U 1 1 579C600A
 P 8695 6115
-F 0 "#PWR057" H 8695 5865 50  0001 C CNN
+F 0 "#PWR048" H 8695 5865 50  0001 C CNN
 F 1 "GNDA" H 8695 5965 50  0000 C CNN
 F 2 "" H 8695 6115 60  0000 C CNN
@@
 $EndComp
 $Comp
-L GND #PWR058
+L GND #PWR049
 U 1 1 579C6010
 P 9015 6115
-F 0 "#PWR058" H 9015 5865 50  0001 C CNN
+F 0 "#PWR049" H 9015 5865 50  0001 C CNN
 F 1 "GND" H 9015 5965 50  0000 C CNN
 F 2 "" H 9015 6115 60  0000 C CNN
@@
 F 0 "JVO60" H 9500 4000 50  0000 C CNN
 F 1 "JUMPER" H 9500 3770 50  0000 C CNN
-F 2 "" H 9500 3850 50  0000 C CNN
+F 2 "CON-SMD-2.54:HARWIN-M20-87-2x1" H 9500 3850 50  0001 C CNN
 F 3 "" H 9500 3850 50  0000 C CNN
 	1    9500 3850
@@
 F 0 "DVO60" V 10200 3650 50  0000 C CNN
 F 1 "BAT54C" V 10300 3650 50  0000 C CNN
-F 2 "" H 10050 3850 50  0000 C CNN
+F 2 "" H 10050 3850 50  0001 C CNN
 F 3 "" H 10050 3850 50  0000 C CNN
 	1    10050 3850
@@
 VGAOUT_R
 $Comp
-L +5V #PWR?
+L +5V #PWR050
 U 1 1 57AD1593
 P 9100 3800
-F 0 "#PWR?" H 9100 3650 50  0001 C CNN
+F 0 "#PWR050" H 9100 3650 50  0001 C CNN
 F 1 "+5V" H 9100 3940 50  0000 C CNN
 F 2 "" H 9100 3800 60  0000 C CNN
@@
 F 0 "CVO61" H 6125 4550 50  0000 L CNN
 F 1 "100nF" H 6125 4350 50  0000 L CNN
-F 2 "" H 6138 4300 50  0000 C CNN
+F 2 "Capacitors_SMD:C_1206_HandSoldering" H 6138 4300 50  0001 C CNN
 F 3 "" H 6100 4450 50  0000 C CNN
 	1    6100 4450
@@
 $EndComp
 $Comp
-L GND #PWR?
+L GND #PWR051
 U 1 1 57AD40D1
 P 6100 4650
-F 0 "#PWR?" H 6100 4400 50  0001 C CNN
+F 0 "#PWR051" H 6100 4400 50  0001 C CNN
 F 1 "GND" H 6100 4500 50  0000 C CNN
 F 2 "" H 6100 4650 60  0000 C CNN
@@
 $EndComp
 $Comp
-L GND #PWR?
+L GND #PWR052
 U 1 1 57AD47F8
 P 6850 6250
-F 0 "#PWR?" H 6850 6000 50  0001 C CNN
+F 0 "#PWR052" H 6850 6000 50  0001 C CNN
 F 1 "GND" H 6850 6100 50  0000 C CNN
 F 2 "" H 6850 6250 60  0000 C CNN
@@
 F 0 "CVO63" H 6125 6150 50  0000 L CNN
 F 1 "100nF" H 6125 5950 50  0000 L CNN
-F 2 "" H 6138 5900 50  0000 C CNN
+F 2 "Capacitors_SMD:C_1206_HandSoldering" H 6138 5900 50  0001 C CNN
 F 3 "" H 6100 6050 50  0000 C CNN
 	1    6100 6050
@@
 $EndComp
 $Comp
-L GND #PWR?
+L GND #PWR053
 U 1 1 57AD4BBD
 P 6100 6250
-F 0 "#PWR?" H 6100 6000 50  0001 C CNN
+F 0 "#PWR053" H 6100 6000 50  0001 C CNN
 F 1 "GND" H 6100 6100 50  0000 C CNN
 F 2 "" H 6100 6250 60  0000 C CNN
@@
 $EndComp
 $Comp
-L GND #PWR?
+L GND #PWR054
 U 1 1 57AD65F2
 P 8700 4150
-F 0 "#PWR?" H 8700 3900 50  0001 C CNN
+F 0 "#PWR054" H 8700 3900 50  0001 C CNN
 F 1 "GND" H 8700 4000 50  0000 C CNN
 F 2 "" H 8700 4150 60  0000 C CNN
@@
 $EndComp
 $Comp
-L +5V #PWR?
+L +5V #PWR055
 U 1 1 57AD7439
 P 6900 4100
-F 0 "#PWR?" H 6900 3950 50  0001 C CNN
+F 0 "#PWR055" H 6900 3950 50  0001 C CNN
 F 1 "+5V" H 6900 4240 50  0000 C CNN
 F 2 "" H 6900 4100 60  0000 C CNN
@@
 F 0 "CVO62" H 7625 4550 50  0000 L CNN
 F 1 "100nF" H 7625 4350 50  0000 L CNN
-F 2 "" H 7638 4300 50  0000 C CNN
+F 2 "Capacitors_SMD:C_1206_HandSoldering" H 7638 4300 50  0001 C CNN
 F 3 "" H 7600 4450 50  0000 C CNN
 	1    7600 4450
@@
 $EndComp
 $Comp
-L GND #PWR?
+L GND #PWR056
 U 1 1 57AD9280
 P 7600 4650
-F 0 "#PWR?" H 7600 4400 50  0001 C CNN
+F 0 "#PWR056" H 7600 4400 50  0001 C CNN
 F 1 "GND" H 7600 4500 50  0000 C CNN
 F 2 "" H 7600 4650 60  0000 C CNN
@@
 F 0 "CVO60" H 10525 4150 50  0000 L CNN
 F 1 "100nF" H 10525 3950 50  0000 L CNN
-F 2 "" H 10538 3900 50  0000 C CNN
+F 2 "Capacitors_SMD:C_1206_HandSoldering" H 10538 3900 50  0001 C CNN
 F 3 "" H 10500 4050 50  0000 C CNN
 	1    10500 4050
@@
 $EndComp
 $Comp
-L GND #PWR?
+L GND #PWR057
 U 1 1 57ADA02C
 P 10700 4300
-F 0 "#PWR?" H 10700 4050 50  0001 C CNN
+F 0 "#PWR057" H 10700 4050 50  0001 C CNN
 F 1 "GND" H 10700 4150 50  0000 C CNN
 F 2 "" H 10700 4300 60  0000 C CNN
@@
 VGAIN_R
 $Comp
-L GNDA #PWR?
+L GNDA #PWR058
 U 1 1 57ADDCDF
 P 9950 3250
-F 0 "#PWR?" H 9950 3000 50  0001 C CNN
+F 0 "#PWR058" H 9950 3000 50  0001 C CNN
 F 1 "GNDA" H 9950 3100 50  0000 C CNN
 F 2 "" H 9950 3250 60  0000 C CNN
@@
 $EndComp
 $Comp
-L GND #PWR?
+L GND #PWR059
 U 1 1 57ADDCE5
 P 4700 2800
-F 0 "#PWR?" H 4700 2550 50  0001 C CNN
+F 0 "#PWR059" H 4700 2550 50  0001 C CNN
 F 1 "GND" V 4700 2600 50  0000 C CNN
 F 2 "" H 4700 2800 60  0000 C CNN
@@
 $EndComp
 $Comp
-L +3V3 #PWR?
+L +3V3 #PWR060
 U 1 1 57ADDD06
 P 5250 1100
-F 0 "#PWR?" H 5250 950 50  0001 C CNN
+F 0 "#PWR060" H 5250 950 50  0001 C CNN
 F 1 "+3V3" H 5250 1240 50  0000 C CNN
 F 2 "" H 5250 1100 60  0000 C CNN
@@
 $EndComp
 $Comp
-L GNDA #PWR?
+L GNDA #PWR061
 U 1 1 57ADDD18
 P 8495 3115
-F 0 "#PWR?" H 8495 2865 50  0001 C CNN
+F 0 "#PWR061" H 8495 2865 50  0001 C CNN
 F 1 "GNDA" H 8495 2965 50  0000 C CNN
 F 2 "" H 8495 3115 60  0000 C CNN
@@
 $EndComp
 $Comp
-L GND #PWR?
+L GND #PWR062
 U 1 1 57ADDD1E
 P 8815 3115
-F 0 "#PWR?" H 8815 2865 50  0001 C CNN
+F 0 "#PWR062" H 8815 2865 50  0001 C CNN
 F 1 "GND" H 8815 2965 50  0000 C CNN
 F 2 "" H 8815 3115 60  0000 C CNN
@@
 F 0 "JVI60" H 9300 1000 50  0000 C CNN
 F 1 "JUMPER" H 9300 770 50  0000 C CNN
-F 2 "" H 9300 850 50  0000 C CNN
+F 2 "CON-SMD-2.54:HARWIN-M20-87-2x1" H 9300 850 50  0001 C CNN
 F 3 "" H 9300 850 50  0000 C CNN
 	1    9300 850
@@
 F 0 "DVI60" V 10000 650 50  0000 C CNN
 F 1 "BAT54C" V 10100 650 50  0000 C CNN
-F 2 "" H 9850 850 50  0000 C CNN
+F 2 "" H 9850 850 50  0001 C CNN
 F 3 "" H 9850 850 50  0000 C CNN
 	1    9850 850
@@
 VGAOUT_R
 $Comp
-L +5V #PWR?
+L +5V #PWR063
 U 1 1 57ADDD42
 P 8900 800
-F 0 "#PWR?" H 8900 650 50  0001 C CNN
+F 0 "#PWR063" H 8900 650 50  0001 C CNN
 F 1 "+5V" H 8900 940 50  0000 C CNN
 F 2 "" H 8900 800 60  0000 C CNN
@@
 F 0 "CVI61" H 5925 1550 50  0000 L CNN
 F 1 "100nF" H 5925 1350 50  0000 L CNN
-F 2 "" H 5938 1300 50  0000 C CNN
+F 2 "Capacitors_SMD:C_1206_HandSoldering" H 5938 1300 50  0001 C CNN
 F 3 "" H 5900 1450 50  0000 C CNN
 	1    5900 1450
@@
 $EndComp
 $Comp
-L GND #PWR?
+L GND #PWR064
 U 1 1 57ADDD54
 P 5900 1650
-F 0 "#PWR?" H 5900 1400 50  0001 C CNN
+F 0 "#PWR064" H 5900 1400 50  0001 C CNN
 F 1 "GND" H 5900 1500 50  0000 C CNN
 F 2 "" H 5900 1650 60  0000 C CNN
@@
 $EndComp
 $Comp
-L GND #PWR?
+L GND #PWR065
 U 1 1 57ADDD5A
 P 6650 3250
-F 0 "#PWR?" H 6650 3000 50  0001 C CNN
+F 0 "#PWR065" H 6650 3000 50  0001 C CNN
 F 1 "GND" H 6650 3100 50  0000 C CNN
 F 2 "" H 6650 3250 60  0000 C CNN
@@
 F 0 "CVI63" H 5925 3150 50  0000 L CNN
 F 1 "100nF" H 5925 2950 50  0000 L CNN
-F 2 "" H 5938 2900 50  0000 C CNN
+F 2 "Capacitors_SMD:C_1206_HandSoldering" H 5938 2900 50  0001 C CNN
 F 3 "" H 5900 3050 50  0000 C CNN
 	1    5900 3050
@@
 $EndComp
 $Comp
-L GND #PWR?
+L GND #PWR066
 U 1 1 57ADDD66
 P 5900 3250
-F 0 "#PWR?" H 5900 3000 50  0001 C CNN
+F 0 "#PWR066" H 5900 3000 50  0001 C CNN
 F 1 "GND" H 5900 3100 50  0000 C CNN
 F 2 "" H 5900 3250 60  0000 C CNN
@@
 $EndComp
 $Comp
-L GND #PWR?
+L GND #PWR067
 U 1 1 57ADDD6C
 P 8500 1150
-F 0 "#PWR?" H 8500 900 50  0001 C CNN
+F 0 "#PWR067" H 8500 900 50  0001 C CNN
 F 1 "GND" H 8500 1000 50  0000 C CNN
 F 2 "" H 8500 1150 60  0000 C CNN
@@
 $EndComp
 $Comp
-L +5V #PWR?
+L +5V #PWR068
 U 1 1 57ADDD72
 P 6700 1100
-F 0 "#PWR?" H 6700 950 50  0001 C CNN
+F 0 "#PWR068" H 6700 950 50  0001 C CNN
 F 1 "+5V" H 6700 1240 50  0000 C CNN
 F 2 "" H 6700 1100 60  0000 C CNN
@@
 F 0 "CVI62" H 7425 1550 50  0000 L CNN
 F 1 "100nF" H 7425 1350 50  0000 L CNN
-F 2 "" H 7438 1300 50  0000 C CNN
+F 2 "Capacitors_SMD:C_1206_HandSoldering" H 7438 1300 50  0001 C CNN
 F 3 "" H 7400 1450 50  0000 C CNN
 	1    7400 1450
@@
 $EndComp
 $Comp
-L GND #PWR?
+L GND #PWR069
 U 1 1 57ADDD84
 P 7400 1650
-F 0 "#PWR?" H 7400 1400 50  0001 C CNN
+F 0 "#PWR069" H 7400 1400 50  0001 C CNN
 F 1 "GND" H 7400 1500 50  0000 C CNN
 F 2 "" H 7400 1650 60  0000 C CNN
@@
 F 0 "CVI60" H 10325 1150 50  0000 L CNN
 F 1 "100nF" H 10325 950 50  0000 L CNN
-F 2 "" H 10338 900 50  0000 C CNN
+F 2 "Capacitors_SMD:C_1206_HandSoldering" H 10338 900 50  0001 C CNN
 F 3 "" H 10300 1050 50  0000 C CNN
 	1    10300 1050
@@
 $EndComp
 $Comp
-L GND #PWR?
+L GND #PWR070
 U 1 1 57ADDDF4
 P 10500 1300
-F 0 "#PWR?" H 10500 1050 50  0001 C CNN
+F 0 "#PWR070" H 10500 1050 50  0001 C CNN
 F 1 "GND" H 10500 1150 50  0000 C CNN
 F 2 "" H 10500 1300 60  0000 C CNN
@@
 Connection ~ 1850 4500
 $Comp
-L +5V #PWR?
+L +5V #PWR071
 U 1 1 57AEA714
 P 2550 2800
-F 0 "#PWR?" H 2550 2650 50  0001 C CNN
+F 0 "#PWR071" H 2550 2650 50  0001 C CNN
 F 1 "+5V" H 2550 2940 50  0000 C CNN
 F 2 "" H 2550 2800 60  0000 C CNN
@@
 F 0 "CVO64" H 5860 6150 50  0000 L CNN
 F 1 "100nF" H 5860 5950 50  0000 L CNN
-F 2 "" H 5873 5900 50  0000 C CNN
+F 2 "Capacitors_SMD:C_1206_HandSoldering" H 5873 5900 50  0001 C CNN
 F 3 "" H 5835 6050 50  0000 C CNN
 	1    5835 6050
@@
 F 0 "CVI64" H 5655 3155 50  0000 L CNN
 F 1 "100nF" H 5655 2955 50  0000 L CNN
-F 2 "" H 5668 2905 50  0000 C CNN
+F 2 "Capacitors_SMD:C_1206_HandSoldering" H 5668 2905 50  0001 C CNN
 F 3 "" H 5630 3055 50  0000 C CNN
 	1    5630 3055

Commit message: Trying to import new netlist.
Parts:
- DVI60, DVO60: footprint (none) -> TO_SOT_Packages_SMD:SOT-23
- UCVI0: footprint SOT23-6 -> TO_SOT_Packages_SMD:SOT-23-6
- UVI_I2C0, UVO_I2C0: footprint SSOP-16 -> Housings_SSOP:SSOP-16_3.9x4.9mm_Pitch0.635mm
Changed lines of the file:
@@
 F 0 "DVO60" V 10200 3650 50  0000 C CNN
 F 1 "BAT54C" V 10300 3650 50  0000 C CNN
-F 2 "" H 10050 3850 50  0001 C CNN
+F 2 "TO_SOT_Packages_SMD:SOT-23" H 10050 3850 50  0001 C CNN
 F 3 "" H 10050 3850 50  0000 C CNN
 	1    10050 3850
@@
 F 0 "UVO_I2C0" H 7150 4300 60  0000 C CNN
 F 1 "TPD7S019" H 7150 4200 60  0000 C CNN
-F 2 "SSOP-16" H 7150 4100 60  0001 C CNN
+F 2 "Housings_SSOP:SSOP-16_3.9x4.9mm_Pitch0.635mm" H 7150 4100 60  0001 C CNN
 F 3 "http://www.ti.com/lit/ds/symlink/tpd7s019.pdf" H 8050 4000 60  0001 C CNN
 	1    6850 5150
@@
 F 0 "DVI60" V 10000 650 50  0000 C CNN
 F 1 "BAT54C" V 10100 650 50  0000 C CNN
-F 2 "" H 9850 850 50  0001 C CNN
+F 2 "TO_SOT_Packages_SMD:SOT-23" H 9850 850 50  0001 C CNN
 F 3 "" H 9850 850 50  0000 C CNN
 	1    9850 850
@@
 F 0 "UVI_I2C0" H 6950 1300 60  0000 C CNN
 F 1 "TPD7S019" H 6950 1200 60  0000 C CNN
-F 2 "SSOP-16" H 6950 1100 60  0001 C CNN
+F 2 "Housings_SSOP:SSOP-16_3.9x4.9mm_Pitch0.635mm" H 6950 1100 60  0001 C CNN
 F 3 "http://www.ti.com/lit/ds/symlink/tpd7s019.pdf" H 7850 1000 60  0001 C CNN
 	1    6650 2150
@@
 F 0 "UCVI0" H 2750 3150 60  0000 C CNN
 F 1 "SP724AH" H 2800 3050 60  0000 C CNN
-F 2 "SOT23-6" H 2550 3050 60  0001 C CNN
+F 2 "TO_SOT_Packages_SMD:SOT-23-6" H 2550 3050 60  0001 C CNN
 F 3 "http://www.littelfuse.com/~/media/electronics/datasheets/tvs_diode_arrays/littelfuse_tvs_diode_array_sp724_datasheet.pdf.pdf" H 3850 2950 60  0001 C CNN
 	1    2550 3750

Commit message: Lots of small fixes to the schematic.
Parts:
- added RVIE1, RVIE2, RVIE3, RVIE4, RVIE5, RVIE6: 0, Resistors_SMD:R_0805_HandSoldering, symbol R
- PVI_I2C3: value VGA Out I2C 3v -> VGA In I2C 3v
- PVI_I2C5: value VGA Out I2C 5v -> VGA In I2C 5v
Connections:
- net GND: now also PVI0.10 (P10), PVI0.5 (P5), PVO0.10 (P10), PVO0.5 (P5)
- net GNDA: no longer PVI0.10 (P10), PVI0.5 (P5), PVO0.10 (P10), PVO0.5 (P5)
- net VGAIN_B: no longer PVO0.3 (P3), UVO_I2C0.3 (Video1)
- net VGAIN_G: no longer PVO0.2 (P2), UVO_I2C0.4 (Video2)
- net VGAIN_HSYNC: now also PVI0.13 (P13), RVIE2.2, RVIE4.1, RVIE4.2, RVIE6.1; no longer UVI_I2C0.15 (SYNC_IN2)
- net VGAIN_R: no longer PVO0.1 (P1), UVO_I2C0.5 (Video3)
- net VGAIN_VSYNC: now also PVI0.14 (P14), RVIE1.2, RVIE3.1, RVIE3.2, RVIE5.1; no longer UVI_I2C0.13 (SYNC_IN1)
- net VGAOUT5V_SCL: no longer PVI0.15 (P15), PVI_I2C5.2 (P2), RVI50.2, UVI_I2C0.9 (DDC_OUT1)
- net VGAOUT5V_SDA: no longer PVI0.12 (P12), PVI_I2C5.3 (P3), RVI51.2, UVI_I2C0.12 (DDC_OUT2)
- net VGAOUT_HSYNC: no longer PVI0.13 (P13), UVI_I2C0.16 (SYNC_OUT2)
- net VGAOUT_VSYNC: no longer PVI0.14 (P14), UVI_I2C0.14 (SYNC_OUT1)
- new net: RVIE1.1, UVI_I2C0.13 (SYNC_IN1)
- new net: RVIE5.2, UVI_I2C0.14 (SYNC_OUT1)
- new net: RVIE2.1, UVI_I2C0.15 (SYNC_IN2)
- new net: RVIE6.2, UVI_I2C0.16 (SYNC_OUT2)
- new net VGAIN5V_SCL: PVI0.15 (P15), PVI_I2C5.2 (P2), RVI50.2, UVI_I2C0.9 (DDC_OUT1)
- new net VGAIN5V_SDA: PVI0.12 (P12), PVI_I2C5.3 (P3), RVI51.2, UVI_I2C0.12 (DDC_OUT2)
- new net VGAOUT_B: PVO0.3 (P3), UVO_I2C0.3 (Video1)
- new net VGAOUT_G: PVO0.2 (P2), UVO_I2C0.4 (Video2)
- new net VGAOUT_R: PVO0.1 (P1), UVO_I2C0.5 (Video3)
Other:
- note added: "Analog"
- note added: "BGND"
- note added: "Digital"
- note added: "GGND"
- note added: "I2CGND\n"
- note added: "Place near \nVGA In\nconnector"
- note added: "Place near \nVGA Out \nconnector"
- note added: "RGND"
- note added: "SYNCGND"
- note removed: "Place near VGA\nOut connector"

Commit message: Fixing the footprint for lots of things.
 * Capacitors 0805 or can.
 * Resistors 0603.
Parts:
- CVI0, CVO0: value C -> 100n; footprint Capacitors_SMD:C_1206_HandSoldering -> Capacitors_SMD:C_0805_HandSoldering
- CVI60, CVI61, CVI62, CVI63, CVI64, CVO60, CVO61, CVO62, CVO63, CVO64: value 100nF -> 100n; footprint Capacitors_SMD:C_1206_HandSoldering -> Capacitors_SMD:C_0805_HandSoldering
- RVI30, RVI31, RVI50, RVI51, RVI60, RVIE1, RVIE2, RVIE3, RVIE4, RVIE5, RVIE6, RVO30, RVO31, RVO50, RVO51, RVO60: footprint Resistors_SMD:R_0805_HandSoldering -> Resistors_SMD:R_0603_HandSoldering
Changed lines of the file:
@@
 F 0 "RVO51" V 8230 4500 50  0000 C CNN
 F 1 "4K7" V 8150 4500 50  0000 C CNN
-F 2 "Resistors_SMD:R_0805_HandSoldering" V 8080 4500 30  0001 C CNN
+F 2 "Resistors_SMD:R_0603_HandSoldering" V 8080 4500 30  0001 C CNN
 F 3 "" H 8150 4500 30  0000 C CNN
 	1    8150 4500
@@
 F 0 "RVO50" V 8030 4500 50  0000 C CNN
 F 1 "4K7" V 7950 4500 50  0000 C CNN
-F 2 "Resistors_SMD:R_0805_HandSoldering" V 7880 4500 30  0001 C CNN
+F 2 "Resistors_SMD:R_0603_HandSoldering" V 7880 4500 30  0001 C CNN
 F 3 "" H 7950 4500 30  0000 C CNN
 	1    7950 4500
@@
 F 0 "RVO31" V 5930 4500 50  0000 C CNN
 F 1 "2K2" V 5850 4500 50  0000 C CNN
-F 2 "Resistors_SMD:R_0805_HandSoldering" V 5780 4500 30  0001 C CNN
+F 2 "Resistors_SMD:R_0603_HandSoldering" V 5780 4500 30  0001 C CNN
 F 3 "" H 5850 4500 30  0000 C CNN
 	1    5850 4500
@@
 F 0 "RVO30" V 5730 4500 50  0000 C CNN
 F 1 "2K2" V 5650 4500 50  0000 C CNN
-F 2 "Resistors_SMD:R_0805_HandSoldering" V 5580 4500 30  0001 C CNN
+F 2 "Resistors_SMD:R_0603_HandSoldering" V 5580 4500 30  0001 C CNN
 F 3 "" H 5650 4500 30  0000 C CNN
 	1    5650 4500
@@
 P 8855 5785
 F 0 "CVO0" H 8880 5885 50  0000 L CNN
-F 1 "C" H 8880 5685 50  0000 L CNN
-F 2 "Capacitors_SMD:C_1206_HandSoldering" H 8893 5635 50  0001 C CNN
+F 1 "100n" H 8880 5685 50  0000 L CNN
+F 2 "Capacitors_SMD:C_0805_HandSoldering" H 8893 5635 50  0001 C CNN
 F 3 "" H 8855 5785 50  0000 C CNN
 	1    8855 5785
@@
 P 6100 4450
 F 0 "CVO61" H 6125 4550 50  0000 L CNN
-F 1 "100nF" H 6125 4350 50  0000 L CNN
-F 2 "Capacitors_SMD:C_1206_HandSoldering" H 6138 4300 50  0001 C CNN
+F 1 "100n" H 6125 4350 50  0000 L CNN
+F 2 "Capacitors_SMD:C_0805_HandSoldering" H 6138 4300 50  0001 C CNN
 F 3 "" H 6100 4450 50  0000 C CNN
 	1    6100 4450
@@
 P 6100 6050
 F 0 "CVO63" H 6125 6150 50  0000 L CNN
-F 1 "100nF" H 6125 5950 50  0000 L CNN
-F 2 "Capacitors_SMD:C_1206_HandSoldering" H 6138 5900 50  0001 C CNN
+F 1 "100n" H 6125 5950 50  0000 L CNN
+F 2 "Capacitors_SMD:C_0805_HandSoldering" H 6138 5900 50  0001 C CNN
 F 3 "" H 6100 6050 50  0000 C CNN
 	1    6100 6050
@@
 F 0 "RVO60" V 10980 4050 50  0000 C CNN
 F 1 "2K2" V 10900 4050 50  0000 C CNN
-F 2 "Resistors_SMD:R_0805_HandSoldering" V 10830 4050 30  0001 C CNN
+F 2 "Resistors_SMD:R_0603_HandSoldering" V 10830 4050 30  0001 C CNN
 F 3 "" H 10900 4050 30  0000 C CNN
 	1    10900 4050
@@
 P 7600 4450
 F 0 "CVO62" H 7625 4550 50  0000 L CNN
-F 1 "100nF" H 7625 4350 50  0000 L CNN
-F 2 "Capacitors_SMD:C_1206_HandSoldering" H 7638 4300 50  0001 C CNN
+F 1 "100n" H 7625 4350 50  0000 L CNN
+F 2 "Capacitors_SMD:C_0805_HandSoldering" H 7638 4300 50  0001 C CNN
 F 3 "" H 7600 4450 50  0000 C CNN
 	1    7600 4450
@@
 P 10500 4050
 F 0 "CVO60" H 10525 4150 50  0000 L CNN
-F 1 "100nF" H 10525 3950 50  0000 L CNN
-F 2 "Capacitors_SMD:C_1206_HandSoldering" H 10538 3900 50  0001 C CNN
+F 1 "100n" H 10525 3950 50  0000 L CNN
+F 2 "Capacitors_SMD:C_0805_HandSoldering" H 10538 3900 50  0001 C CNN
 F 3 "" H 10500 4050 50  0000 C CNN
 	1    10500 4050
@@
 F 0 "RVI51" V 8030 1500 50  0000 C CNN
 F 1 "4K7" V 7950 1500 50  0000 C CNN
-F 2 "Resistors_SMD:R_0805_HandSoldering" V 7880 1500 30  0001 C CNN
+F 2 "Resistors_SMD:R_0603_HandSoldering" V 7880 1500 30  0001 C CNN
 F 3 "" H 7950 1500 30  0000 C CNN
 	1    7950 1500
@@
 F 0 "RVI50" V 7830 1500 50  0000 C CNN
 F 1 "4K7" V 7750 1500 50  0000 C CNN
-F 2 "Resistors_SMD:R_0805_HandSoldering" V 7680 1500 30  0001 C CNN
+F 2 "Resistors_SMD:R_0603_HandSoldering" V 7680 1500 30  0001 C CNN
 F 3 "" H 7750 1500 30  0000 C CNN
 	1    7750 1500
@@
 F 0 "RVI31" V 5730 1500 50  0000 C CNN
 F 1 "2K2" V 5650 1500 50  0000 C CNN
-F 2 "Resistors_SMD:R_0805_HandSoldering" V 5580 1500 30  0001 C CNN
+F 2 "Resistors_SMD:R_0603_HandSoldering" V 5580 1500 30  0001 C CNN
 F 3 "" H 5650 1500 30  0000 C CNN
 	1    5650 1500
@@
 F 0 "RVI30" V 5530 1500 50  0000 C CNN
 F 1 "2K2" V 5450 1500 50  0000 C CNN
-F 2 "Resistors_SMD:R_0805_HandSoldering" V 5380 1500 30  0001 C CNN
+F 2 "Resistors_SMD:R_0603_HandSoldering" V 5380 1500 30  0001 C CNN
 F 3 "" H 5450 1500 30  0000 C CNN
 	1    5450 1500
@@
 P 8655 2785
 F 0 "CVI0" H 8680 2885 50  0000 L CNN
-F 1 "C" H 8680 2685 50  0000 L CNN
-F 2 "Capacitors_SMD:C_1206_HandSoldering" H 8693 2635 50  0001 C CNN
+F 1 "100n" H 8680 2685 50  0000 L CNN
+F 2 "Capacitors_SMD:C_0805_HandSoldering" H 8693 2635 50  0001 C CNN
 F 3 "" H 8655 2785 50  0000 C CNN
 	1    8655 2785
@@
 P 5900 1450
 F 0 "CVI61" H 5925 1550 50  0000 L CNN
-F 1 "100nF" H 5925 1350 50  0000 L CNN
-F 2 "Capacitors_SMD:C_1206_HandSoldering" H 5938 1300 50  0001 C CNN
+F 1 "100n" H 5925 1350 50  0000 L CNN
+F 2 "Capacitors_SMD:C_0805_HandSoldering" H 5938 1300 50  0001 C CNN
 F 3 "" H 5900 1450 50  0000 C CNN
 	1    5900 1450
@@
 P 5900 3050
 F 0 "CVI63" H 5925 3150 50  0000 L CNN
-F 1 "100nF" H 5925 2950 50  0000 L CNN
-F 2 "Capacitors_SMD:C_1206_HandSoldering" H 5938 2900 50  0001 C CNN
+F 1 "100n" H 5925 2950 50  0000 L CNN
+F 2 "Capacitors_SMD:C_0805_HandSoldering" H 5938 2900 50  0001 C CNN
 F 3 "" H 5900 3050 50  0000 C CNN
 	1    5900 3050
@@
 F 0 "RVI60" V 10780 1050 50  0000 C CNN
 F 1 "2K2" V 10700 1050 50  0000 C CNN
-F 2 "Resistors_SMD:R_0805_HandSoldering" V 10630 1050 30  0001 C CNN
+F 2 "Resistors_SMD:R_0603_HandSoldering" V 10630 1050 30  0001 C CNN
 F 3 "" H 10700 1050 30  0000 C CNN
 	1    10700 1050
@@
 P 7400 1450
 F 0 "CVI62" H 7425 1550 50  0000 L CNN
-F 1 "100nF" H 7425 1350 50  0000 L CNN
-F 2 "Capacitors_SMD:C_1206_HandSoldering" H 7438 1300 50  0001 C CNN
+F 1 "100n" H 7425 1350 50  0000 L CNN
+F 2 "Capacitors_SMD:C_0805_HandSoldering" H 7438 1300 50  0001 C CNN
 F 3 "" H 7400 1450 50  0000 C CNN
 	1    7400 1450
@@
 P 10300 1050
 F 0 "CVI60" H 10325 1150 50  0000 L CNN
-F 1 "100nF" H 10325 950 50  0000 L CNN
-F 2 "Capacitors_SMD:C_1206_HandSoldering" H 10338 900 50  0001 C CNN
+F 1 "100n" H 10325 950 50  0000 L CNN
+F 2 "Capacitors_SMD:C_0805_HandSoldering" H 10338 900 50  0001 C CNN
 F 3 "" H 10300 1050 50  0000 C CNN
 	1    10300 1050
@@
 P 5835 6050
 F 0 "CVO64" H 5860 6150 50  0000 L CNN
-F 1 "100nF" H 5860 5950 50  0000 L CNN
-F 2 "Capacitors_SMD:C_1206_HandSoldering" H 5873 5900 50  0001 C CNN
+F 1 "100n" H 5860 5950 50  0000 L CNN
+F 2 "Capacitors_SMD:C_0805_HandSoldering" H 5873 5900 50  0001 C CNN
 F 3 "" H 5835 6050 50  0000 C CNN
 	1    5835 6050
@@
 P 5630 3055
 F 0 "CVI64" H 5655 3155 50  0000 L CNN
-F 1 "100nF" H 5655 2955 50  0000 L CNN
-F 2 "Capacitors_SMD:C_1206_HandSoldering" H 5668 2905 50  0001 C CNN
+F 1 "100n" H 5655 2955 50  0000 L CNN
+F 2 "Capacitors_SMD:C_0805_HandSoldering" H 5668 2905 50  0001 C CNN
 F 3 "" H 5630 3055 50  0000 C CNN
 	1    5630 3055
@@
 F 0 "RVIE5" V 8100 2200 50  0000 C CNN
 F 1 "0" V 8100 2200 50  0001 C CNN
-F 2 "Resistors_SMD:R_0805_HandSoldering" V 8030 2200 30  0001 C CNN
+F 2 "Resistors_SMD:R_0603_HandSoldering" V 8030 2200 30  0001 C CNN
 F 3 "" H 8100 2200 30  0000 C CNN
 	1    8100 2200
@@
 F 0 "RVIE6" V 8100 2300 50  0000 C CNN
 F 1 "0" V 8100 2300 50  0001 C CNN
-F 2 "Resistors_SMD:R_0805_HandSoldering" V 8030 2300 30  0001 C CNN
+F 2 "Resistors_SMD:R_0603_HandSoldering" V 8030 2300 30  0001 C CNN
 F 3 "" H 8100 2300 30  0000 C CNN
 	1    8100 2300
@@
 F 0 "RVIE3" V 7575 2150 50  0000 C CNN
 F 1 "0" V 7575 2150 50  0001 C CNN
-F 2 "Resistors_SMD:R_0805_HandSoldering" V 7505 2150 30  0001 C CNN
+F 2 "Resistors_SMD:R_0603_HandSoldering" V 7505 2150 30  0001 C CNN
 F 3 "" H 7575 2150 30  0000 C CNN
 	1    7575 2150
@@
 F 0 "RVIE4" V 7575 2250 50  0000 C CNN
 F 1 "0" V 7575 2250 50  0001 C CNN
-F 2 "Resistors_SMD:R_0805_HandSoldering" V 7505 2250 30  0001 C CNN
+F 2 "Resistors_SMD:R_0603_HandSoldering" V 7505 2250 30  0001 C CNN
 F 3 "" H 7575 2250 30  0000 C CNN
 	1    7575 2250
@@
 F 0 "RVIE1" V 5775 2200 50  0000 C CNN
 F 1 "0" V 5775 2200 50  0001 C CNN
-F 2 "Resistors_SMD:R_0805_HandSoldering" V 5705 2200 30  0001 C CNN
+F 2 "Resistors_SMD:R_0603_HandSoldering" V 5705 2200 30  0001 C CNN
 F 3 "" H 5775 2200 30  0000 C CNN
 	1    5775 2200
@@
 F 0 "RVIE2" V 5775 2300 50  0000 C CNN
 F 1 "0" V 5775 2300 50  0001 C CNN
-F 2 "Resistors_SMD:R_0805_HandSoldering" V 5705 2300 30  0001 C CNN
+F 2 "Resistors_SMD:R_0603_HandSoldering" V 5705 2300 30  0001 C CNN
 F 3 "" H 5775 2300 30  0000 C CNN
 	1    5775 2300
