File: board/ad9984.sch (KiCad schematic (older format))
At the start: 40 parts, among them P401 AD9984 I2C, U401 AD9984

Commit message: Annotate.
Parts:
- gave numbers to parts that had none: 1
Changed lines of the file:
@@
 R[0..9]
 $Comp
-L GNDA #PWR022
+L GNDA #PWR23
 U 1 1 5640DDDC
 P 4200 5050
-F 0 "#PWR022" H 4200 4800 50  0001 C CNN
+F 0 "#PWR23" H 4200 4800 50  0001 C CNN
 F 1 "GNDA" H 4200 4900 50  0000 C CNN
 F 2 "" H 4200 5050 60  0000 C CNN
@@
 VGA_R
 $Comp
-L +3.3V #PWR026
+L +3.3V #PWR35
 U 1 1 56413478
 P 7850 5250
-F 0 "#PWR026" H 7850 5100 50  0001 C CNN
+F 0 "#PWR35" H 7850 5100 50  0001 C CNN
 F 1 "+3.3V" V 7860 5470 50  0000 C CNN
 F 2 "" H 7850 5250 60  0000 C CNN
@@
 $EndComp
 $Comp
-L +3.3V #PWR028
+L +3.3V #PWR25
 U 1 1 56413584
 P 5900 5250
-F 0 "#PWR028" H 5900 5100 50  0001 C CNN
+F 0 "#PWR25" H 5900 5100 50  0001 C CNN
 F 1 "+3.3V" H 5900 5400 50  0000 C CNN
 F 2 "" H 5900 5250 60  0000 C CNN
@@
 $EndComp
 $Comp
-L VD #PWR029
+L VD #PWR24
 U 1 1 564135D1
 P 5150 2850
-F 0 "#PWR029" H 5150 2700 50  0001 C CNN
+F 0 "#PWR24" H 5150 2700 50  0001 C CNN
 F 1 "VD" H 5150 2990 50  0000 C CNN
 F 2 "" H 5150 2850 60  0000 C CNN
@@
 	5900 6150 5900 6250
 $Comp
-L GND #PWR030
+L GND #PWR26
 U 1 1 5641452A
 P 5900 6250
-F 0 "#PWR030" H 5900 6000 50  0001 C CNN
+F 0 "#PWR26" H 5900 6000 50  0001 C CNN
 F 1 "GND" H 5900 6100 50  0000 C CNN
 F 2 "" H 5900 6250 60  0000 C CNN
@@
 Connection ~ 3750 4950
 $Comp
-L GND #PWR031
+L GND #PWR31
 U 1 1 56415296
 P 6750 5350
-F 0 "#PWR031" H 6750 5100 50  0001 C CNN
+F 0 "#PWR31" H 6750 5100 50  0001 C CNN
 F 1 "GND" V 6750 5150 50  0000 C CNN
 F 2 "" H 6750 5350 60  0000 C CNN
@@
 $EndComp
 $Comp
-L GND #PWR032
+L GND #PWR36
 U 1 1 5641579B
 P 8000 5250
-F 0 "#PWR032" H 8000 5000 50  0001 C CNN
+F 0 "#PWR36" H 8000 5000 50  0001 C CNN
 F 1 "GND" H 8000 5100 50  0000 C CNN
 F 2 "" H 8000 5250 60  0000 C CNN
@@
 DATACK
 $Comp
-L PVD #PWR033
+L PVD #PWR29
 U 1 1 56415C22
 P 6550 2250
-F 0 "#PWR033" H 6550 2100 50  0001 C CNN
+F 0 "#PWR29" H 6550 2100 50  0001 C CNN
 F 1 "PVD" H 6550 2390 50  0000 C CNN
 F 2 "" H 6550 2250 60  0000 C CNN
@@
 	7150 2450 7150 2250
 $Comp
-L GND #PWR034
+L GND #PWR27
 U 1 1 564164E1
 P 6000 2350
-F 0 "#PWR034" H 6000 2100 50  0001 C CNN
+F 0 "#PWR27" H 6000 2100 50  0001 C CNN
 F 1 "GND" V 5900 2300 50  0000 C CNN
 F 2 "" H 6000 2350 60  0000 C CNN
@@
 Connection ~ 6150 2350
 $Comp
-L VD #PWR035
+L VD #PWR38
 U 1 1 56416F9D
 P 8950 4750
-F 0 "#PWR035" H 8950 4600 50  0001 C CNN
+F 0 "#PWR38" H 8950 4600 50  0001 C CNN
 F 1 "VD" V 9000 4750 50  0000 C CNN
 F 2 "" H 8950 4750 60  0000 C CNN
@@
 $EndComp
 $Comp
-L GND #PWR036
+L GND #PWR39
 U 1 1 564170A0
 P 9000 3550
-F 0 "#PWR036" H 9000 3300 50  0001 C CNN
+F 0 "#PWR39" H 9000 3300 50  0001 C CNN
 F 1 "GND" V 9050 3600 50  0000 C CNN
 F 2 "" H 9000 3550 60  0000 C CNN
@@
 $EndComp
 $Comp
-L GND #PWR037
+L GND #PWR32
 U 1 1 564172D9
 P 6900 1200
-F 0 "#PWR037" H 6900 950 50  0001 C CNN
+F 0 "#PWR32" H 6900 950 50  0001 C CNN
 F 1 "GND" H 6900 1050 50  0000 C CNN
 F 2 "" H 6900 1200 60  0000 C CNN
@@
 $EndComp
 $Comp
-L PVD #PWR038
+L PVD #PWR28
 U 1 1 56417326
 P 6350 1200
-F 0 "#PWR038" H 6350 1050 50  0001 C CNN
+F 0 "#PWR28" H 6350 1050 50  0001 C CNN
 F 1 "PVD" H 6350 1340 50  0000 C CNN
 F 2 "" H 6350 1200 60  0000 C CNN
@@
 $EndComp
 $Comp
-L GND #PWR039
+L GND #PWR33
 U 1 1 5655A202
 P 7300 1800
-F 0 "#PWR039" H 7300 1550 50  0001 C CNN
+F 0 "#PWR33" H 7300 1550 50  0001 C CNN
 F 1 "GND" H 7250 1650 50  0000 C CNN
 F 2 "" H 7300 1800 60  0000 C CNN
@@
 $EndComp
 $Comp
-L GND #PWR040
+L GND #PWR37
 U 1 1 5692FBEE
 P 8250 1850
-F 0 "#PWR040" H 8250 1600 50  0001 C CNN
+F 0 "#PWR37" H 8250 1600 50  0001 C CNN
 F 1 "GND" V 8250 1650 50  0000 C CNN
 F 2 "" H 8250 1850 50  0000 C CNN
@@
 Connection ~ 8050 2050
 $Comp
-L GNDA #PWR?
+L GNDA #PWR21
 U 1 1 57976F35
 P 3680 5980
-F 0 "#PWR?" H 3680 5730 50  0001 C CNN
+F 0 "#PWR21" H 3680 5730 50  0001 C CNN
 F 1 "GNDA" H 3680 5830 50  0000 C CNN
 F 2 "" H 3680 5980 60  0000 C CNN
@@
 $EndComp
 $Comp
-L GND #PWR?
+L GND #PWR22
 U 1 1 57976FB5
 P 4000 5980
-F 0 "#PWR?" H 4000 5730 50  0001 C CNN
+F 0 "#PWR22" H 4000 5730 50  0001 C CNN
 F 1 "GND" H 4000 5830 50  0000 C CNN
 F 2 "" H 4000 5980 60  0000 C CNN
@@
 $EndComp
 $Comp
-L C C?
+L C C1
 U 1 1 5797716F
 P 3840 5650
-F 0 "C?" H 3865 5750 50  0000 L CNN
+F 0 "C1" H 3865 5750 50  0000 L CNN
 F 1 "C" H 3865 5550 50  0000 L CNN
 F 2 "" H 3878 5500 50  0000 C CNN
@@
 	4000 5980 4000 5650
 $Comp
-L +3.3V #PWR?
+L +3.3V #PWR34
 U 1 1 5796E857
 P 7500 1200
-F 0 "#PWR?" H 7500 1050 50  0001 C CNN
+F 0 "#PWR34" H 7500 1050 50  0001 C CNN
 F 1 "+3.3V" H 7500 1340 50  0000 C CNN
 F 2 "" H 7500 1200 50  0000 C CNN
@@
 Connection ~ 7550 1250
 $Comp
-L +3.3V #PWR?
+L +3.3V #PWR30
 U 1 1 5796EFF3
 P 6650 5350
-F 0 "#PWR?" H 6650 5200 50  0001 C CNN
+F 0 "#PWR30" H 6650 5200 50  0001 C CNN
 F 1 "+3.3V" V 6660 5570 50  0000 C CNN
 F 2 "" H 6650 5350 60  0000 C CNN
@@
 $EndComp
 $Comp
-L +3.3V #PWR?
+L +3.3V #PWR40
 U 1 1 5796F1FD
 P 9100 3650
-F 0 "#PWR?" H 9100 3500 50  0001 C CNN
+F 0 "#PWR40" H 9100 3500 50  0001 C CNN
 F 1 "+3.3V" V 9110 3870 50  0000 C CNN
 F 2 "" H 9100 3650 60  0000 C CNN

Commit message: Lots of small fixes.
Other:
- note added: "Analog VGA Signals\nNoise sensitive!"
Changed lines of the file:
@@
 $Descr A4 11693 8268
 encoding utf-8
-Sheet 4 6
+Sheet 4 5
 Title "TOFE VGA Expansion Board - AD9984"
 Date "2015-11-25"
@@
 Text Notes 3870 2340 0    60   ~ 0
 1V8 - VD - Analog side 1V8 supply\n1V8 - PVD - Digital side 1V8 supply\n3V3 - +3.3V - IO Level
+Wire Notes Line
+	4620 2500 6020 2500
+Wire Notes Line
+	6020 2500 6020 4970
+Wire Notes Line
+	6020 4970 5550 4970
+Wire Notes Line
+	5550 4970 5550 6310
+Wire Notes Line
+	5550 6310 1270 6310
+Wire Notes Line
+	1270 6310 1270 2500
+Wire Notes Line
+	1270 2500 4610 2500
+Text Notes 1360 2710 0    60   ~ 0
+Analog VGA Signals\nNoise sensitive!
 Wire Wire Line
 	4000 5650 3990 5650

Commit message: Adding new parts.
Parts:
- C1: footprint (none) -> Capacitors_SMD:C_0805_HandSoldering
Changed lines of the file:
@@
 F 0 "C1" H 3865 5750 50  0000 L CNN
 F 1 "C" H 3865 5550 50  0000 L CNN
-F 2 "" H 3878 5500 50  0000 C CNN
+F 2 "Capacitors_SMD:C_0805_HandSoldering" H 3878 5500 50  0001 C CNN
 F 3 "" H 3840 5650 50  0000 C CNN
 	1    3840 5650
