File: board/TOFE-VGA.sch (KiCad schematic (older format))
At the start: 1 part, among them P1 CONN_02X06

Commit message: Updating net names.
Changed lines of the file:
@@
 F3 "G[0..9]" I L 6550 4020 60
 F4 "B[0..9]" I L 6550 4120 60
-F5 "SCL_VGA_TX" B R 9250 4300 60
-F6 "SDA_VGA_TX" B R 9250 4200 60
-F7 "SCL_VGA_RX" B R 9250 4700 60
-F8 "SDA_VGA_RX" B R 9250 4600 60
+F5 "VGAIN_SDA" B R 9250 4300 60
+F6 "VGAIN_SCL" B R 9250 4200 60
+F7 "VGAOUT_SDA" B R 9250 4700 60
+F8 "VGAOUT_SCL" B R 9250 4600 60
 F9 "SDA_AD9984" B L 6550 4850 60
 F10 "SCL_AD9984" B L 6550 4950 60
@@
 F13 "SOGOUT" I L 6550 4600 60
 F14 "DATACK" B L 6550 4700 60
-F15 "EN_VGA_TX" O R 9250 4900 60
-F16 "EN_VGA_RX" O R 9250 5000 60
+F15 "VGAOUT_I2C_EN" O R 9250 4900 60
+F16 "VGAIN_I2C_EN" O R 9250 5000 60
 F17 "RST" O L 6550 5100 60
 F18 "FIELD" I L 6550 4305 60
@@
 F0 "TOFE-VGA/VGA" 50
 F1 "vga.sch" 50
-F2 "SCL_VGA_RX" B R 7000 2500 60
-F3 "SDA_VGA_RX" B R 7000 2600 60
-F4 "SCL_VGA_TX" B R 7000 2750 60
-F5 "SDA_VGA_TX" B R 7000 2850 60
+F2 "VGAOUT_SCL" B R 7000 2500 60
+F3 "VGAOUT_SDA" B R 7000 2600 60
+F4 "VGAIN_SCL" B R 7000 2750 60
+F5 "VGAIN_SDA" B R 7000 2850 60
 F6 "VGAIN_B" O L 5100 2605 60
 F7 "VGAIN_G" O L 5100 2505 60
@@
 F9 "VGAIN_HSYNC0" O L 5100 2305 60
 F10 "VGAIN_VSYNC0" O L 5100 2205 60
-F11 "EN_VGA_RX" I R 7000 2250 60
-F12 "EN_VGA_TX" I R 7000 2350 60
+F11 "VGAIN_I2C_EN" I R 7000 2250 60
+F12 "VGAOUT_I2C_EN" I R 7000 2350 60
 F13 "COMP_Y" O L 5100 3385 60
 F14 "COMP_Pb" O L 5100 3485 60
@@
 $EndComp
 $Comp
-L GND #PWR01
+L GND #PWR1
 U 1 1 579D1C68
 P 5015 3215
-F 0 "#PWR01" H 5015 2965 50  0001 C CNN
+F 0 "#PWR1" H 5015 2965 50  0001 C CNN
 F 1 "GND" H 5015 3065 50  0000 C CNN
 F 2 "" H 5015 3215 50  0000 C CNN

Commit message: ERC and removing 0 from vsync/hsync.
Connections:
- net TOFE-VGA/AD9984/HSYNC0 renamed TOFE-VGA/AD9984/VGA_HSYNC
- net TOFE-VGA/AD9984/VSYNC0 renamed TOFE-VGA/AD9984/VGA_VSYNC
- net TOFE-VGA/VGA/VGAOUT_HSYNC0 renamed TOFE-VGA/VGA/VGAOUT_HSYNC
- net TOFE-VGA/VGA/VGAOUT_VSYNC0 renamed TOFE-VGA/VGA/VGAOUT_VSYNC
Changed lines of the file:
@@
 F9 "SOGOUT" O R 5550 4600 60
 F10 "DATACK" B R 5550 4700 60
-F11 "VSYNC0" I L 3200 4650 60
-F12 "HSYNC0" I L 3200 4550 60
+F11 "VGA_VSYNC" I L 3200 4650 60
+F12 "VGA_HSYNC" I L 3200 4550 60
 F13 "SDA_AD9984" B R 5550 4850 60
 F14 "SCL_AD9984" B R 5550 4950 60
@@
 F7 "VGAIN_G" O L 5100 2505 60
 F8 "VGAIN_R" O L 5100 2405 60
-F9 "VGAIN_HSYNC0" O L 5100 2305 60
-F10 "VGAIN_VSYNC0" O L 5100 2205 60
+F9 "VGAIN_HSYNC" O L 5100 2305 60
+F10 "VGAIN_VSYNC" O L 5100 2205 60
 F11 "VGAIN_I2C_EN" I R 7000 2250 60
 F12 "VGAOUT_I2C_EN" I R 7000 2350 60
@@
 F17 "VGAOUT_G" I L 5100 3015 60
 F18 "VGAOUT_R" I L 5100 2915 60
-F19 "VGAOUT_HSYNC0" I L 5100 2815 60
-F20 "VGAOUT_VSYNC0" I L 5100 2715 60
+F19 "VGAOUT_HSYNC" I L 5100 2815 60
+F20 "VGAOUT_VSYNC" I L 5100 2715 60
 $EndSheet
 $Comp

Commit message: Lots of small fixes to the schematic.
Parts:
- renumbered P1 to PJVGA1
Changed lines of the file:
@@
 F13 "SOGOUT" I L 6550 4600 60
 F14 "DATACK" B L 6550 4700 60
-F15 "VGAOUT_I2C_EN" O R 9250 4900 60
-F16 "VGAIN_I2C_EN" O R 9250 5000 60
 F17 "RST" O L 6550 5100 60
 F18 "FIELD" I L 6550 4305 60
@@
 F9 "VGAIN_HSYNC" O L 5100 2305 60
 F10 "VGAIN_VSYNC" O L 5100 2205 60
-F11 "VGAIN_I2C_EN" I R 7000 2250 60
-F12 "VGAOUT_I2C_EN" I R 7000 2350 60
 F13 "COMP_Y" O L 5100 3385 60
 F14 "COMP_Pb" O L 5100 3485 60
@@
 $EndSheet
 $Comp
-L CONN_02X06 P1
+L CONN_02X06 PJVGA1
 U 1 1 579CCE5F
 P 4725 2965
-F 0 "P1" H 4725 3315 50  0000 C CNN
-F 1 "CONN_02X06" H 4725 2615 50  0000 C CNN
+F 0 "PJVGA1" H 4725 2605 50  0000 C CNN
+F 1 "CONN_02X06" H 4725 2615 50  0001 C CNN
 F 2 "Pin_Headers:Pin_Header_Straight_2x06" H 4725 1765 50  0001 C CNN
 F 3 "" H 4725 1765 50  0000 C CNN
@@
 	5550 4700 6550 4700
 Wire Wire Line
-	7000 2350 10000 2350
-Wire Wire Line
-	10000 2350 10000 4900
-Wire Wire Line
-	10000 4900 9250 4900
-Wire Wire Line
-	9250 5000 10100 5000
-Wire Wire Line
-	10100 5000 10100 2250
-Wire Wire Line
-	10100 2250 7000 2250
-Wire Wire Line
 	2370 5050 2370 3585
 Wire Wire Line
@@
 Wire Wire Line
 	5550 5100 6550 5100
+Text Label 7600 2500 0    60   ~ 0
+VGAOUT_SCL
+Text Label 7600 2600 0    60   ~ 0
+VGAOUT_SDA
+Text Label 7600 2750 0    60   ~ 0
+VGAIN_SCL
+Text Label 7600 2850 0    60   ~ 0
+VGAIN_SDA
+Text Label 5910 3920 0    60   ~ 0
+R[0..9]
+Text Label 5910 4020 0    60   ~ 0
+G[0..9]
+Text Label 5910 4120 0    60   ~ 0
+B[0..9]
+Text Label 5935 4305 0    60   ~ 0
+FIELD
+Text Label 5936 4400 0    60   ~ 0
+VSOUT
+Text Label 5934 4500 0    60   ~ 0
+HSOUT
+Text Label 5934 4600 0    60   ~ 0
+SOGOUT
+Text Label 5929 4700 0    60   ~ 0
+DATACK
+Text Label 5771 4850 0    60   ~ 0
+SDA_AD9984
+Text Label 5771 4950 0    60   ~ 0
+SCL_AD99844
+Text Label 5983 5100 0    60   ~ 0
+RST
 $EndSCHEMATC
