File: board/power.sch (KiCad schematic (older format))
At the start: 38 parts, among them U5V1 LP2985

Commit message: Small updates from review by RattusRattus.
Parts:
- C5VI2: renamed from C215; value C5VI2 -> 10n
- C5VO1: value 2u2 -> 22u
- renumbered CIO1 to CAIO1, CIO2 to CAIO2, CIO3 to CAIO3, CIO4 to CI2C1, CIO5 to CI2C2
Other:
- note added: "Place CAIO* near AD9984 pins\nPlace CI2C1 near UVI_I2C0\nPlace CI2C2 near UVO_I2C0\nPlace *TIO* near TOFE pins"
- note removed: "Place CIO* near AD9984 pins\nPlace *TIO* near TOFE pins"
Changed lines of the file:
@@
 P 8650 2250
 F 0 "C5VO1" H 8675 2350 50  0000 L CNN
-F 1 "2u2" H 8675 2150 50  0000 L CNN
+F 1 "22u" H 8675 2150 50  0000 L CNN
 F 2 "Capacitors_SMD:c_elec_4x5.8" H 8688 2100 30  0001 C CNN
 F 3 "" H 8650 2250 60  0000 C CNN
@@
 $EndComp
 $Comp
-L C C215
+L C C5VI2
 U 1 1 56425EF8
 P 6800 2750
-F 0 "C215" H 6825 2850 50  0000 L CNN
-F 1 "C5VI2" H 6825 2650 50  0000 L CNN
+F 0 "C5VI2" H 6825 2850 50  0000 L CNN
+F 1 "10n" H 6825 2650 50  0000 L CNN
 F 2 "Resistors_SMD:R_0805_HandSoldering" H 6838 2600 30  0001 C CNN
 F 3 "" H 6800 2750 60  0000 C CNN
@@
 $EndComp
 $Comp
-L C CIO1
+L C CAIO1
 U 1 1 56932788
 P 3800 2500
-F 0 "CIO1" H 3825 2600 50  0000 L CNN
+F 0 "CAIO1" H 3825 2600 50  0000 L CNN
 F 1 "100n" H 3825 2400 50  0000 L CNN
 F 2 "Resistors_SMD:R_0805_HandSoldering" H 3838 2350 30  0001 C CNN
@@
 $EndComp
 $Comp
-L C CIO2
+L C CAIO2
 U 1 1 5693278E
 P 4050 2500
-F 0 "CIO2" H 4075 2600 50  0000 L CNN
+F 0 "CAIO2" H 4075 2600 50  0000 L CNN
 F 1 "100n" H 4075 2400 50  0000 L CNN
 F 2 "Resistors_SMD:R_0805_HandSoldering" H 4088 2350 30  0001 C CNN
@@
 $EndComp
 $Comp
-L C CIO3
+L C CAIO3
 U 1 1 56932794
 P 4300 2500
-F 0 "CIO3" H 4325 2600 50  0000 L CNN
+F 0 "CAIO3" H 4325 2600 50  0000 L CNN
 F 1 "100n" H 4325 2400 50  0000 L CNN
 F 2 "Resistors_SMD:R_0805_HandSoldering" H 4338 2350 30  0001 C CNN
@@
 $EndComp
 $Comp
-L C CIO4
+L C CI2C1
 U 1 1 5693279A
 P 4550 2500
-F 0 "CIO4" H 4575 2600 50  0000 L CNN
+F 0 "CI2C1" H 4575 2600 50  0000 L CNN
 F 1 "100n" H 4575 2400 50  0000 L CNN
 F 2 "Resistors_SMD:R_0805_HandSoldering" H 4588 2350 30  0001 C CNN
@@
 $EndComp
 $Comp
-L C CIO5
+L C CI2C2
 U 1 1 569327A0
 P 4800 2500
-F 0 "CIO5" H 4825 2600 50  0000 L CNN
+F 0 "CI2C2" H 4825 2600 50  0000 L CNN
 F 1 "100n" H 4825 2400 50  0000 L CNN
 F 2 "Resistors_SMD:R_0805_HandSoldering" H 4838 2350 30  0001 C CNN
@@
 Text Notes 3325 4225 0    60   ~ 0
 Place CVD* near AD9984 pins\nPlace others near UVD1
-Text Notes 3715 1960 0    60   ~ 0
-Place CIO* near AD9984 pins\nPlace *TIO* near TOFE pins
+Text Notes 3655 1680 0    60   ~ 0
+Place CAIO* near AD9984 pins\nPlace CI2C1 near UVI_I2C0\nPlace CI2C2 near UVO_I2C0\nPlace *TIO* near TOFE pins
 Text Notes 6970 1710 0    60   ~ 0
 Place all *5V* componets near each other

Commit message: Lots of small fixes to the schematic.
Parts:
- removed CI2C1, CI2C2: 100n, Resistors_SMD:R_0805_HandSoldering, symbol C
Other:
- note added: "Place CAIO* near AD9984 pins\nPlace *TIO* near TOFE pins"
- note removed: "Place CAIO* near AD9984 pins\nPlace CI2C1 near UVI_I2C0\nPlace CI2C2 near UVO_I2C0\nPlace *TIO* near TOFE pins"
Changed lines of the file:
@@
-	1    0    0    -1
-$EndComp
-$Comp
-L C CI2C1
-U 1 1 5693279A
-P 4550 2500
-F 0 "CI2C1" H 4575 2600 50  0000 L CNN
-F 1 "100n" H 4575 2400 50  0000 L CNN
-F 2 "Resistors_SMD:R_0805_HandSoldering" H 4588 2350 30  0001 C CNN
-F 3 "" H 4550 2500 60  0000 C CNN
-	1    4550 2500
-	1    0    0    -1
-$EndComp
-$Comp
-L C CI2C2
-U 1 1 569327A0
-P 4800 2500
-F 0 "CI2C2" H 4825 2600 50  0000 L CNN
-F 1 "100n" H 4825 2400 50  0000 L CNN
-F 2 "Resistors_SMD:R_0805_HandSoldering" H 4838 2350 30  0001 C CNN
-F 3 "" H 4800 2500 60  0000 C CNN
-	1    4800 2500
 	1    0    0    -1
 $EndComp
@@
 	4300 2050 4300 2350
 Connection ~ 4300 2050
-Wire Wire Line
-	4550 2050 4550 2350
-Connection ~ 4550 2050
-Wire Wire Line
-	4550 2650 4550 2950
-Connection ~ 4550 2950
-Wire Wire Line
-	4800 2950 4800 2650
-Wire Wire Line
-	4800 2050 4800 2350
-Connection ~ 4800 2050
 $Comp
 L R RTIO1
@@
 Wire Wire Line
 	5200 2950 5200 2900
-Connection ~ 4800 2950
 Wire Wire Line
 	3450 2000 3450 2050
@@
 Place CVD* near AD9984 pins\nPlace others near UVD1
 Text Notes 3655 1680 0    60   ~ 0
-Place CAIO* near AD9984 pins\nPlace CI2C1 near UVI_I2C0\nPlace CI2C2 near UVO_I2C0\nPlace *TIO* near TOFE pins
+Place CAIO* near AD9984 pins\nPlace *TIO* near TOFE pins
 Text Notes 6970 1710 0    60   ~ 0
 Place all *5V* componets near each other

Commit message: Fixing the footprint for lots of things.
 * Capacitors 0805 or can.
 * Resistors 0603.
Parts:
- C5VI1: value 1u -> 22u
- C5VI2, CAIO1, CAIO2, CAIO3, CPV1, CPV2, CPV3, CVD1, CVD2, CVD3, CVD4, CVD5: footprint Resistors_SMD:R_0805_HandSoldering -> Capacitors_SMD:C_0805_HandSoldering
- R12V1, R5V1, RPV1, RPV2, RPV3, RTIO1, RVD1, RVD2, RVD3: footprint Resistors_SMD:R_0805_HandSoldering -> Resistors_SMD:R_0603_HandSoldering
Changed lines of the file:
@@
 F 0 "RVD2" V 3530 4750 50  0000 C CNN
 F 1 "147K" V 3450 4750 50  0000 C CNN
-F 2 "Resistors_SMD:R_0805_HandSoldering" V 3380 4750 30  0001 C CNN
+F 2 "Resistors_SMD:R_0603_HandSoldering" V 3380 4750 30  0001 C CNN
 F 3 "" H 3450 4750 30  0000 C CNN
 	1    3450 4750
@@
 F 0 "RVD1" V 3280 4400 50  0000 C CNN
 F 1 "76K8" V 3200 4400 50  0000 C CNN
-F 2 "Resistors_SMD:R_0805_HandSoldering" V 3130 4400 30  0001 C CNN
+F 2 "Resistors_SMD:R_0603_HandSoldering" V 3130 4400 30  0001 C CNN
 F 3 "" H 3200 4400 30  0000 C CNN
 	1    3200 4400
@@
 F 0 "CVD1" H 3975 4850 50  0000 L CNN
 F 1 "100n" H 3975 4650 50  0000 L CNN
-F 2 "Resistors_SMD:R_0805_HandSoldering" H 3988 4600 30  0001 C CNN
+F 2 "Capacitors_SMD:C_0805_HandSoldering" H 3988 4600 30  0001 C CNN
 F 3 "" H 3950 4750 60  0000 C CNN
 	1    3950 4750
@@
 F 0 "CVD2" H 4225 4850 50  0000 L CNN
 F 1 "100n" H 4225 4650 50  0000 L CNN
-F 2 "Resistors_SMD:R_0805_HandSoldering" H 4238 4600 30  0001 C CNN
+F 2 "Capacitors_SMD:C_0805_HandSoldering" H 4238 4600 30  0001 C CNN
 F 3 "" H 4200 4750 60  0000 C CNN
 	1    4200 4750
@@
 F 0 "CVD3" H 4475 4850 50  0000 L CNN
 F 1 "100n" H 4475 4650 50  0000 L CNN
-F 2 "Resistors_SMD:R_0805_HandSoldering" H 4488 4600 30  0001 C CNN
+F 2 "Capacitors_SMD:C_0805_HandSoldering" H 4488 4600 30  0001 C CNN
 F 3 "" H 4450 4750 60  0000 C CNN
 	1    4450 4750
@@
 F 0 "CVD4" H 4725 4850 50  0000 L CNN
 F 1 "100n" H 4725 4650 50  0000 L CNN
-F 2 "Resistors_SMD:R_0805_HandSoldering" H 4738 4600 30  0001 C CNN
+F 2 "Capacitors_SMD:C_0805_HandSoldering" H 4738 4600 30  0001 C CNN
 F 3 "" H 4700 4750 60  0000 C CNN
 	1    4700 4750
@@
 F 0 "CVD5" H 4975 4850 50  0000 L CNN
 F 1 "100n" H 4975 4650 50  0000 L CNN
-F 2 "Resistors_SMD:R_0805_HandSoldering" H 4988 4600 30  0001 C CNN
+F 2 "Capacitors_SMD:C_0805_HandSoldering" H 4988 4600 30  0001 C CNN
 F 3 "" H 4950 4750 60  0000 C CNN
 	1    4950 4750
@@
 F 0 "RPV2" V 8680 4750 50  0000 C CNN
 F 1 "147K" V 8600 4750 50  0000 C CNN
-F 2 "Resistors_SMD:R_0805_HandSoldering" V 8530 4750 30  0001 C CNN
+F 2 "Resistors_SMD:R_0603_HandSoldering" V 8530 4750 30  0001 C CNN
 F 3 "" H 8600 4750 30  0000 C CNN
 	1    8600 4750
@@
 F 0 "RPV1" V 8430 4400 50  0000 C CNN
 F 1 "76K8" V 8350 4400 50  0000 C CNN
-F 2 "Resistors_SMD:R_0805_HandSoldering" V 8280 4400 30  0001 C CNN
+F 2 "Resistors_SMD:R_0603_HandSoldering" V 8280 4400 30  0001 C CNN
 F 3 "" H 8350 4400 30  0000 C CNN
 	1    8350 4400
@@
 F 0 "CPV1" H 9125 4850 50  0000 L CNN
 F 1 "100n" H 9125 4650 50  0000 L CNN
-F 2 "Resistors_SMD:R_0805_HandSoldering" H 9138 4600 30  0001 C CNN
+F 2 "Capacitors_SMD:C_0805_HandSoldering" H 9138 4600 30  0001 C CNN
 F 3 "" H 9100 4750 60  0000 C CNN
 	1    9100 4750
@@
 F 0 "CPV2" H 9375 4850 50  0000 L CNN
 F 1 "100n" H 9375 4650 50  0000 L CNN
-F 2 "Resistors_SMD:R_0805_HandSoldering" H 9388 4600 30  0001 C CNN
+F 2 "Capacitors_SMD:C_0805_HandSoldering" H 9388 4600 30  0001 C CNN
 F 3 "" H 9350 4750 60  0000 C CNN
 	1    9350 4750
@@
 F 0 "CPV3" H 9625 4850 50  0000 L CNN
 F 1 "100n" H 9625 4650 50  0000 L CNN
-F 2 "Resistors_SMD:R_0805_HandSoldering" H 9638 4600 30  0001 C CNN
+F 2 "Capacitors_SMD:C_0805_HandSoldering" H 9638 4600 30  0001 C CNN
 F 3 "" H 9600 4750 60  0000 C CNN
 	1    9600 4750
@@
 F 0 "C5VI2" H 6825 2850 50  0000 L CNN
 F 1 "10n" H 6825 2650 50  0000 L CNN
-F 2 "Resistors_SMD:R_0805_HandSoldering" H 6838 2600 30  0001 C CNN
+F 2 "Capacitors_SMD:C_0805_HandSoldering" H 6838 2600 30  0001 C CNN
 F 3 "" H 6800 2750 60  0000 C CNN
 	1    6800 2750
@@
 P 6600 2250
 F 0 "C5VI1" H 6625 2350 50  0000 L CNN
-F 1 "1u" H 6625 2150 50  0000 L CNN
+F 1 "22u" H 6625 2150 50  0000 L CNN
 F 2 "Capacitors_SMD:c_elec_4x5.8" H 6638 2100 30  0001 C CNN
 F 3 "" H 6600 2250 60  0000 C CNN
@@
 F 0 "R12V1" H 2650 2750 50  0000 C CNN
 F 1 "470R" V 2450 2750 50  0000 C CNN
-F 2 "Resistors_SMD:R_0805_HandSoldering" V 2380 2750 50  0001 C CNN
+F 2 "Resistors_SMD:R_0603_HandSoldering" V 2380 2750 50  0001 C CNN
 F 3 "" H 2450 2750 50  0000 C CNN
 	1    2450 2750
@@
 F 0 "R5V1" H 9200 2700 50  0000 C CNN
 F 1 "150R" V 9050 2700 50  0000 C CNN
-F 2 "Resistors_SMD:R_0805_HandSoldering" V 8980 2700 50  0001 C CNN
+F 2 "Resistors_SMD:R_0603_HandSoldering" V 8980 2700 50  0001 C CNN
 F 3 "" H 9050 2700 50  0000 C CNN
 	1    9050 2700
@@
 F 0 "RVD3" H 5500 5000 50  0000 C CNN
 F 1 "1R8" V 5350 5000 50  0000 C CNN
-F 2 "Resistors_SMD:R_0805_HandSoldering" V 5280 5000 50  0001 C CNN
+F 2 "Resistors_SMD:R_0603_HandSoldering" V 5280 5000 50  0001 C CNN
 F 3 "" H 5350 5000 50  0000 C CNN
 	1    5350 5000
@@
 F 0 "RPV3" H 10100 5000 50  0000 C CNN
 F 1 "1R8" V 9950 5000 50  0000 C CNN
-F 2 "Resistors_SMD:R_0805_HandSoldering" V 9880 5000 50  0001 C CNN
+F 2 "Resistors_SMD:R_0603_HandSoldering" V 9880 5000 50  0001 C CNN
 F 3 "" H 9950 5000 50  0000 C CNN
 	1    9950 5000
@@
 F 0 "CAIO1" H 3825 2600 50  0000 L CNN
 F 1 "100n" H 3825 2400 50  0000 L CNN
-F 2 "Resistors_SMD:R_0805_HandSoldering" H 3838 2350 30  0001 C CNN
+F 2 "Capacitors_SMD:C_0805_HandSoldering" H 3838 2350 30  0001 C CNN
 F 3 "" H 3800 2500 60  0000 C CNN
 	1    3800 2500
@@
 F 0 "CAIO2" H 4075 2600 50  0000 L CNN
 F 1 "100n" H 4075 2400 50  0000 L CNN
-F 2 "Resistors_SMD:R_0805_HandSoldering" H 4088 2350 30  0001 C CNN
+F 2 "Capacitors_SMD:C_0805_HandSoldering" H 4088 2350 30  0001 C CNN
 F 3 "" H 4050 2500 60  0000 C CNN
 	1    4050 2500
@@
 F 0 "CAIO3" H 4325 2600 50  0000 L CNN
 F 1 "100n" H 4325 2400 50  0000 L CNN
-F 2 "Resistors_SMD:R_0805_HandSoldering" H 4338 2350 30  0001 C CNN
+F 2 "Capacitors_SMD:C_0805_HandSoldering" H 4338 2350 30  0001 C CNN
 F 3 "" H 4300 2500 60  0000 C CNN
 	1    4300 2500
@@
 F 0 "RTIO1" H 5350 2750 50  0000 C CNN
 F 1 "68R" V 5200 2750 50  0000 C CNN
-F 2 "Resistors_SMD:R_0805_HandSoldering" V 5130 2750 50  0001 C CNN
+F 2 "Resistors_SMD:R_0603_HandSoldering" V 5130 2750 50  0001 C CNN
 F 3 "" H 5200 2750 50  0000 C CNN
 	1    5200 2750
