File: board/TOFE-VGA.kicad_pcb (KiCad board)
At the start: 4 copper layers, 46 x 3 mm, 143 parts, among them P1 CONN_02X06, P601 3-RCA, U5V1 LP2985

Commit message: Lots of small fixes.
Parts:
- removed C215: C5VI2, Resistors_SMD:R_0805_HandSoldering
- removed CI2C1, CI2C2, CIO1, CIO2, CIO3, CIO4, CIO5: 100n, Resistors_SMD:R_0805_HandSoldering
- removed D304: LED, LEDs:LED_0805
- removed P1: CONN_02X06, Pin_Headers:Pin_Header_Straight_2x06
- removed R306: 68R, Resistors_SMD:R_0805_HandSoldering
- removed RVI32, RVI34, RVO32, RVO33: ?, Resistors_SMD:R_0805_HandSoldering
- removed TP402: TESTPOINT, 2MM-TESTPOINT:2MM-TESTPOINT
- added DDG4: LED, LEDs:LED_0805, F.Cu at (206.9, 83.4)
- added PJVGA1: CONN_02X06, Pin_Headers:Pin_Header_Straight_2x06, F.Cu at (68.8, 107.2)
- added RDG4: 68R, Resistors_SMD:R_0805_HandSoldering, F.Cu at (199.5, 86.9)
- added RVIE1: 0, Resistors_SMD:R_0805_HandSoldering, F.Cu at (206.7, 88.4)
- added RVIE2: 0, Resistors_SMD:R_0805_HandSoldering, F.Cu at (199.2, 92.9)
- added RVIE3: 0, Resistors_SMD:R_0805_HandSoldering, F.Cu at (213.0, 82.7)
- added RVIE4: 0, Resistors_SMD:R_0805_HandSoldering, F.Cu at (213.2, 85.7)
- added RVIE5: 0, Resistors_SMD:R_0805_HandSoldering, F.Cu at (213.1, 90.2)
- added RVIE6: 0, Resistors_SMD:R_0805_HandSoldering, F.Cu at (211.6, 93.7)
- PDG0: footprint Pin_Headers:Pin_Header_Straight_2x05 -> Pin_Headers:Pin_Header_Straight_2x06
- PVI_I2C3: value VGA Out I2C 3v -> VGA In I2C 3v
- PVI_I2C5: value VGA Out I2C 5v -> VGA In I2C 5v
- moved P601 50.5 mm to (131.4, 49.7)
Connections:
- net /TOFE-VGA/AD9984/DATACK renamed /DATACK
- net /TOFE-VGA/AD9984/FIELD renamed /FIELD
- net /TOFE-VGA/AD9984/HSOUT renamed /HSOUT
- net /TOFE-VGA/AD9984/RST renamed /RST
- net /TOFE-VGA/AD9984/SCL_AD9984 renamed /SCL_AD99844
- net /TOFE-VGA/AD9984/SDA_AD9984 renamed /SDA_AD9984
- net /TOFE-VGA/AD9984/SOGOUT renamed /SOGOUT
- net /TOFE-VGA/AD9984/VSOUT renamed /VSOUT
- net /TOFE-VGA/TOFE/VGAIN_I2C_EN renamed Net-(PDG0-Pad3)
- net /TOFE-VGA/TOFE/VGAIN_SCL renamed /VGAIN_SDA
- net /TOFE-VGA/TOFE/VGAOUT_I2C_EN renamed Net-(PDG0-Pad5)
- net /TOFE-VGA/TOFE/VGAOUT_SCL renamed /VGAOUT_SDA
- net /TOFE-VGA/VGA/VGAIN_SCL renamed /VGAIN_SCL
- net /TOFE-VGA/VGA/VGAOUT_SCL renamed /VGAOUT_SCL
- PDG0 pad 1: Net-(PDG0-Pad1) -> /TOFE-VGA/TOFE/IDDAT
- PDG0 pad 2: +3V3 -> Net-(PDG0-Pad2)
- PDG0 pad 9: Net-(PDG0-Pad9) -> GND
- PVI0 pad 10: GNDA -> GND
- PVI0 pad 11: Net-(PVI0-Pad11) -> (no net)
- PVI0 pad 12: /TOFE-VGA/VGA/VGAOUT5V_SDA -> /TOFE-VGA/VGA/VGAIN5V_SDA
- PVI0 pad 13: /TOFE-VGA/VGA/VGAOUT_HSYNC -> /TOFE-VGA/VGA/VGAIN_HSYNC
- PVI0 pad 14: /TOFE-VGA/VGA/VGAOUT_VSYNC -> /TOFE-VGA/VGA/VGAIN_VSYNC
- PVI0 pad 15: /TOFE-VGA/VGA/VGAOUT5V_SCL -> /TOFE-VGA/VGA/VGAIN5V_SCL
- PVI0 pad 4: Net-(PVI0-Pad4) -> (no net)
- PVI0 pad 5: GNDA -> GND
- PVI_I2C5 pad 2: /TOFE-VGA/VGA/VGAOUT5V_SCL -> /TOFE-VGA/VGA/VGAIN5V_SCL
- PVI_I2C5 pad 3: /TOFE-VGA/VGA/VGAOUT5V_SDA -> /TOFE-VGA/VGA/VGAIN5V_SDA
- PVO0 pad 1: /TOFE-VGA/VGA/VGAIN_R -> /TOFE-VGA/VGA/VGAOUT_R
- PVO0 pad 10: GNDA -> GND
- PVO0 pad 11: Net-(PVO0-Pad11) -> (no net)
- PVO0 pad 2: /TOFE-VGA/VGA/VGAIN_G -> /TOFE-VGA/VGA/VGAOUT_G
- PVO0 pad 3: /TOFE-VGA/VGA/VGAIN_B -> /TOFE-VGA/VGA/VGAOUT_B
- PVO0 pad 4: Net-(PVO0-Pad4) -> (no net)
- PVO0 pad 5: GNDA -> GND
- RDG1 pad 2: Net-(PDG0-Pad4) -> Net-(PDG0-Pad2)
- RDG2 pad 2: Net-(PDG0-Pad6) -> Net-(PDG0-Pad4)
- RDG3 pad 2: Net-(PDG0-Pad8) -> Net-(PDG0-Pad6)
- RVI50 pad 2: /TOFE-VGA/VGA/VGAOUT5V_SCL -> /TOFE-VGA/VGA/VGAIN5V_SCL
- RVI51 pad 2: /TOFE-VGA/VGA/VGAOUT5V_SDA -> /TOFE-VGA/VGA/VGAIN5V_SDA
- TOFE0 pad A33: Net-(TOFE0-PadA33) -> (no net)
- TOFE0 pad B17: Net-(TOFE0-PadB17) -> (no net)
- TOFE0 pad B31: Net-(TOFE0-PadB31) -> (no net)
- UAD9984 pad 19: Net-(UAD9984-Pad19) -> (no net)
- UCVI0 pad 6: Net-(UCVI0-Pad6) -> (no net)
- UPV1 pad 8: Net-(UPV1-Pad8) -> (no net)
- UVD1 pad 8: Net-(UVD1-Pad8) -> (no net)
- UVI_I2C0 pad 12: /TOFE-VGA/VGA/VGAOUT5V_SDA -> /TOFE-VGA/VGA/VGAIN5V_SDA
- UVI_I2C0 pad 13: /TOFE-VGA/VGA/VGAIN_VSYNC -> Net-(RVIE1-Pad1)
- UVI_I2C0 pad 14: /TOFE-VGA/VGA/VGAOUT_VSYNC -> Net-(RVIE5-Pad2)
- UVI_I2C0 pad 15: /TOFE-VGA/VGA/VGAIN_HSYNC -> Net-(RVIE2-Pad1)
- UVI_I2C0 pad 16: /TOFE-VGA/VGA/VGAOUT_HSYNC -> Net-(RVIE6-Pad2)
- UVI_I2C0 pad 9: /TOFE-VGA/VGA/VGAOUT5V_SCL -> /TOFE-VGA/VGA/VGAIN5V_SCL
- UVO_I2C0 pad 3: /TOFE-VGA/VGA/VGAIN_B -> /TOFE-VGA/VGA/VGAOUT_B
- UVO_I2C0 pad 4: /TOFE-VGA/VGA/VGAIN_G -> /TOFE-VGA/VGA/VGAOUT_G
- UVO_I2C0 pad 5: /TOFE-VGA/VGA/VGAIN_R -> /TOFE-VGA/VGA/VGAOUT_R
Routing:
- net /TOFE-VGA/VGA/VGAOUT5V_SCL: track 79.4 -> 32.4 mm
- net /TOFE-VGA/VGA/VGAIN5V_SCL: track 0.00 -> 46.9 mm
- net /TOFE-VGA/VGA/VGAOUT_HSYNC: track 51.0 -> 4.69 mm
- net /TOFE-VGA/VGA/VGAIN_HSYNC: track 108.9 -> 155.2 mm
- net /TOFE-VGA/VGA/VGAIN5V_SDA: track 0.00 -> 41.4 mm
- net /TOFE-VGA/VGA/VGAOUT5V_SDA: track 80.0 -> 38.6 mm
- net /TOFE-VGA/VGA/VGAOUT_VSYNC: track 49.2 -> 22.8 mm
- net /TOFE-VGA/VGA/VGAIN_VSYNC: track 106.2 -> 131.8 mm
- net GNDA: track 97.1 -> 75.9 mm
- net (no net): track 73.2 -> 89.1 mm, vias 4 -> 11
- net GND: track 176.2 -> 190.0 mm, vias 57 -> 52
- net Net-(TP402-Pad1): track 7.28 -> 0.00 mm
- net /FIELD: track 1.61 -> 8.89 mm
- net /TOFE-VGA/VGA/VGAIN_R: track 81.3 -> 75.4 mm, vias 2 -> 1
- net /TOFE-VGA/VGA/VGAOUT_R: track 0.00 -> 5.84 mm, vias 0 -> 1
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
Commit message: Import and update netlist.
Parts:
- removed C1: C, Capacitors_SMD:C_1206_HandSoldering
- added CGND1: 100n, Capacitors_SMD:C_0805_HandSoldering, F.Cu at (174.0, 96.6)
- C301, C410, C411, C5VI2, CAIO1, CAIO2, CAIO3, CCB1, CCR1, CCY1, CCY2, CPV1, CPV2, CPV3, CREF1, CVB1, CVD1, CVD2, CVD3, CVD4, CVD5, CVG1, CVG2, CVR2: footprint Resistors_SMD:R_0805_HandSoldering -> Capacitors_SMD:C_0805_HandSoldering
- C5VI1: value 1u -> 22u
- CVI0, CVO0: value C -> 100n; footprint Capacitors_SMD:C_1206_HandSoldering -> Capacitors_SMD:C_0805_HandSoldering
- CVI60, CVI61, CVI62, CVI63, CVI64, CVO60, CVO61, CVO62, CVO63, CVO64: value 100nF -> 100n; footprint Capacitors_SMD:C_1206_HandSoldering -> Capacitors_SMD:C_0805_HandSoldering
- R12V1, R301, R302, R303, R410, R411, R412, R413, R414, R415, R416, R5V1, RA1, RA2, RCB1, RCR1, RCY1, RDG1, RDG2, RDG3, RDG4, RPV1, RPV2, RPV3, RPWD1, RTIO1, RVB1, RVD1, RVD2, RVD3, RVG1, RVI30, RVI31, RVI50, RVI51, RVI60, RVIE1, RVIE2, RVIE3, RVIE4, RVIE5, RVIE6, RVO30, RVO31, RVO50, RVO51, RVO60, RVR1: footprint Resistors_SMD:R_0805_HandSoldering -> Resistors_SMD:R_0603_HandSoldering
Connections:
- PJVGA1 pad 11: (no net) -> Net-(PJVGA1-Pad11)
- PVI0 pad 11: (no net) -> Net-(PVI0-Pad11)
- PVI0 pad 4: (no net) -> Net-(PVI0-Pad4)
- PVO0 pad 11: (no net) -> Net-(PVO0-Pad11)
- PVO0 pad 4: (no net) -> Net-(PVO0-Pad4)
- TOFE0 pad A33: (no net) -> Net-(TOFE0-PadA33)
- TOFE0 pad B17: (no net) -> Net-(TOFE0-PadB17)
- TOFE0 pad B31: (no net) -> Net-(TOFE0-PadB31)
- UAD9984 pad 19: (no net) -> Net-(UAD9984-Pad19)
- UCVI0 pad 6: (no net) -> Net-(UCVI0-Pad6)
- UPV1 pad 8: (no net) -> Net-(UPV1-Pad8)
- UVD1 pad 8: (no net) -> Net-(UVD1-Pad8)
Routing:
- net (no net): track 89.1 -> 92.0 mm, vias 11 -> 13
- net /TOFE-VGA/VGA/VGAOUT_VSYNC: track 22.8 -> 24.3 mm
- net /TOFE-VGA/VGA/VGAOUT5V_SCL: track 32.4 -> 30.9 mm
- net GNDA: track 75.9 -> 74.4 mm, vias 30 -> 29
- net GND: track 190.0 -> 188.5 mm, vias 52 -> 51
- net Net-(RVIE1-Pad1): track 0.00 -> 1.25 mm
- net /TOFE-VGA/VGA/VGAIN5V_SCL: track 46.9 -> 45.7 mm

Commit message: Updated PCB from Phyllis.
Parts:
- removed CGND1: 100n, Capacitors_SMD:C_0805_HandSoldering
- removed DDG4: LED, LEDs:LED_0805
- removed PJVGA1: CONN_02X06, Pin_Headers:Pin_Header_Straight_2x06
- removed RDG4: 68R, Resistors_SMD:R_0603_HandSoldering
- removed RVIE1, RVIE2, RVIE3, RVIE4, RVIE5, RVIE6: 0, Resistors_SMD:R_0603_HandSoldering
- removed the TOFE0 at (62.2, 154.0)
- added C1: C, Capacitors_SMD:C_1206_HandSoldering, F.Cu at (57.4, 105.8)
- added C215: C5VI2, Resistors_SMD:R_0805_HandSoldering, F.Cu at (83.8, 159.1)
- added CI2C1: 100n, Resistors_SMD:R_0805_HandSoldering, B.Cu at (38.1, 86.7)
- added CI2C2: 100n, Resistors_SMD:R_0805_HandSoldering, B.Cu at (38.1, 108.1)
- added CIO1: 100n, Resistors_SMD:R_0805_HandSoldering, F.Cu at (115.0, 141.9)
- added CIO2: 100n, Resistors_SMD:R_0805_HandSoldering, F.Cu at (90.5, 162.3)
- added CIO3: 100n, Resistors_SMD:R_0805_HandSoldering, F.Cu at (94.1, 162.4)
- added CIO4: 100n, Resistors_SMD:R_0805_HandSoldering, F.Cu at (97.5, 162.4)
- added CIO5: 100n, Resistors_SMD:R_0805_HandSoldering, F.Cu at (101.2, 162.6)
- added D304: LED, LEDs:LED_0805, F.Cu at (143.2, 131.2)
- added P1: CONN_02X06, Pin_Headers:Pin_Header_Straight_2x06, F.Cu at (91.7, 91.0)
- added R306: 68R, Resistors_SMD:R_0805_HandSoldering, F.Cu at (143.2, 135.4)
- added RVI32: ?, Resistors_SMD:R_0805_HandSoldering, F.Cu at (120.7, 144.4)
- added RVI34: ?, Resistors_SMD:R_0805_HandSoldering, F.Cu at (120.7, 146.4)
- added RVO32: ?, Resistors_SMD:R_0805_HandSoldering, F.Cu at (125.3, 144.4)
- added RVO33: ?, Resistors_SMD:R_0805_HandSoldering, F.Cu at (125.3, 146.4)
- added TOFE0 (x2): TOFE-8X, TOFE_8X_HalfHeight:TOFE_8X_HalfHeight, F.Cu at (62.2, 154.0)
- added TP402: TESTPOINT, 2MM-TESTPOINT:2MM-TESTPOINT, F.Cu at (124.8, 126.0)
- C301, C410, C411, C5VI2, CCB1, CCR1, CCY1, CCY2, CPV1, CPV2, CPV3, CVB1, CVD1, CVG1, CVG2, CVR2: footprint Capacitors_SMD:C_0805_HandSoldering -> Resistors_SMD:R_0805_HandSoldering
- C5VI1: value 22u -> 1u
- CAIO1, CAIO2, CAIO3, CREF1, CVD2, CVD3, CVD4, CVD5: footprint Capacitors_SMD:C_0805_HandSoldering -> Resistors_SMD:R_0805_HandSoldering; moved to B.Cu
- CVI0, CVO0: value 100n -> C; footprint Capacitors_SMD:C_0805_HandSoldering -> Capacitors_SMD:C_1206_HandSoldering
- CVI60, CVI61, CVI62, CVO60, CVO61, CVO62: value 100n -> 100nF; footprint Capacitors_SMD:C_0805_HandSoldering -> Capacitors_SMD:C_1206_HandSoldering; moved to B.Cu
- CVI63, CVI64, CVO63, CVO64: value 100n -> 100nF; footprint Capacitors_SMD:C_0805_HandSoldering -> Capacitors_SMD:C_1206_HandSoldering
- DVI60, DVO60, LCR1, LCY1, LVG1, LVR1: moved to B.Cu
- PDG0: footprint Pin_Headers:Pin_Header_Straight_2x06 -> Pin_Headers:Pin_Header_Straight_2x05
- PVI_I2C3: value VGA In I2C 3v -> VGA Out I2C 3v
- PVI_I2C5: value VGA In I2C 5v -> VGA Out I2C 5v
- R12V1, R301, R302, R303, R410, R411, R412, R413, R414, R415, R416, R5V1, RA1, RA2, RCB1, RDG1, RDG2, RDG3, RPV1, RPV2, RPV3, RPWD1, RTIO1, RVB1, RVD1, RVD2, RVD3: footprint Resistors_SMD:R_0603_HandSoldering -> Resistors_SMD:R_0805_HandSoldering
- RCR1, RCY1, RVG1, RVI30, RVI31, RVI50, RVI51, RVI60, RVO30, RVO31, RVO50, RVO51, RVO60, RVR1: footprint Resistors_SMD:R_0603_HandSoldering -> Resistors_SMD:R_0805_HandSoldering; moved to B.Cu
- moved CVI62 152.4 mm to (39.0, 102.9)
- moved CVO62 142.2 mm to (39.0, 81.5)
- moved CVI61 139.2 mm to (39.0, 105.8)
- moved CVO63 136.5 mm to (39.0, 90.5)
- moved CVO61 135.1 mm to (39.0, 84.5)
- moved CVI63 133.8 mm to (38.8, 112.1)
- moved C5VI2 129.3 mm to (86.8, 135.0), turned to 270 degrees
- moved CVO64 123.5 mm to (39.0, 88.1)
- moved CVI64 119.9 mm to (38.8, 109.6)
- moved CVI60 115.4 mm to (82.5, 123.3)
- moved RVI60 111.7 mm to (81.5, 117.6)
- moved DVO60 103.9 mm to (80.7, 77.8), turned to 270 degrees
- moved DVI60 102.4 mm to (80.7, 120.4), turned to 270 degrees
- moved RVO60 101.0 mm to (81.4, 75.1)
- moved CVO60 98.4 mm to (82.4, 80.9)
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Connections:
- net /RST renamed /TOFE-VGA/AD9984/RST
- net /SCL_AD99844 renamed /TOFE-VGA/AD9984/SCL_AD9984
- net /SDA_AD9984 renamed /TOFE-VGA/AD9984/SDA_AD9984
- net /VGAIN_SCL renamed /TOFE-VGA/VGA/VGAIN_SCL
- net /VGAIN_SDA renamed /TOFE-VGA/TOFE/VGAIN_SCL
- net /VGAOUT_SCL renamed /TOFE-VGA/VGA/VGAOUT_SCL
- net /VGAOUT_SDA renamed /TOFE-VGA/TOFE/VGAOUT_SCL
- net /VSOUT renamed /TOFE-VGA/AD9984/VSOUT
- PDG0 pad 1: /TOFE-VGA/TOFE/IDDAT -> Net-(PDG0-Pad1)
- PDG0 pad 2: Net-(PDG0-Pad2) -> +3V3
- PDG0 pad 3: Net-(PDG0-Pad3) -> /TOFE-VGA/TOFE/VGAIN_I2C_EN
- PDG0 pad 5: Net-(PDG0-Pad5) -> /TOFE-VGA/TOFE/VGAOUT_I2C_EN
- PDG0 pad 9: GND -> Net-(PDG0-Pad9)
- PVI0 pad 10: GND -> GNDA
- PVI0 pad 12: /TOFE-VGA/VGA/VGAIN5V_SDA -> /TOFE-VGA/VGA/VGAOUT5V_SDA
- PVI0 pad 13: /TOFE-VGA/VGA/VGAIN_HSYNC -> /TOFE-VGA/VGA/VGAOUT_HSYNC
- PVI0 pad 14: /TOFE-VGA/VGA/VGAIN_VSYNC -> /TOFE-VGA/VGA/VGAOUT_VSYNC
- PVI0 pad 15: /TOFE-VGA/VGA/VGAIN5V_SCL -> /TOFE-VGA/VGA/VGAOUT5V_SCL
- PVI0 pad 5: GND -> GNDA
- PVI_I2C5 pad 2: /TOFE-VGA/VGA/VGAIN5V_SCL -> /TOFE-VGA/VGA/VGAOUT5V_SCL
- PVI_I2C5 pad 3: /TOFE-VGA/VGA/VGAIN5V_SDA -> /TOFE-VGA/VGA/VGAOUT5V_SDA
- PVO0 pad 1: /TOFE-VGA/VGA/VGAOUT_R -> /TOFE-VGA/VGA/VGAIN_R
- PVO0 pad 10: GND -> GNDA
- PVO0 pad 2: /TOFE-VGA/VGA/VGAOUT_G -> /TOFE-VGA/VGA/VGAIN_G
- PVO0 pad 3: /TOFE-VGA/VGA/VGAOUT_B -> /TOFE-VGA/VGA/VGAIN_B
- PVO0 pad 5: GND -> GNDA
- RDG1 pad 2: Net-(PDG0-Pad2) -> Net-(PDG0-Pad4)
- RDG2 pad 2: Net-(PDG0-Pad4) -> Net-(PDG0-Pad6)
- RDG3 pad 2: Net-(PDG0-Pad6) -> Net-(PDG0-Pad8)
- RVI50 pad 2: /TOFE-VGA/VGA/VGAIN5V_SCL -> /TOFE-VGA/VGA/VGAOUT5V_SCL
- RVI51 pad 2: /TOFE-VGA/VGA/VGAIN5V_SDA -> /TOFE-VGA/VGA/VGAOUT5V_SDA
- UAD9984 pad 21: /FIELD -> /TOFE-VGA/AD9984/FIELD
- UAD9984 pad 23: /HSOUT -> /TOFE-VGA/AD9984/HSOUT
- UAD9984 pad 24: /SOGOUT -> /TOFE-VGA/AD9984/SOGOUT
- UAD9984 pad 25: /DATACK -> /TOFE-VGA/AD9984/DATACK
- UVI_I2C0 pad 12: /TOFE-VGA/VGA/VGAIN5V_SDA -> /TOFE-VGA/VGA/VGAOUT5V_SDA
- UVI_I2C0 pad 13: Net-(RVIE1-Pad1) -> /TOFE-VGA/VGA/VGAIN_VSYNC
- UVI_I2C0 pad 14: Net-(RVIE5-Pad2) -> /TOFE-VGA/VGA/VGAOUT_VSYNC
- UVI_I2C0 pad 15: Net-(RVIE2-Pad1) -> /TOFE-VGA/VGA/VGAIN_HSYNC
- UVI_I2C0 pad 16: Net-(RVIE6-Pad2) -> /TOFE-VGA/VGA/VGAOUT_HSYNC
- UVI_I2C0 pad 9: /TOFE-VGA/VGA/VGAIN5V_SCL -> /TOFE-VGA/VGA/VGAOUT5V_SCL
- UVO_I2C0 pad 3: /TOFE-VGA/VGA/VGAOUT_B -> /TOFE-VGA/VGA/VGAIN_B
- UVO_I2C0 pad 4: /TOFE-VGA/VGA/VGAOUT_G -> /TOFE-VGA/VGA/VGAIN_G
- UVO_I2C0 pad 5: /TOFE-VGA/VGA/VGAOUT_R -> /TOFE-VGA/VGA/VGAIN_R
Routing:
- net /TOFE-VGA/VGA/VGAIN_HSYNC: track 155.2 -> 33.1 mm
- net /TOFE-VGA/TOFE/VGAOUT_SCL: track 187.7 -> 80.1 mm, vias 2 -> 0
- net /TOFE-VGA/VGA/VGAIN_VSYNC: track 131.8 -> 32.5 mm
- net /TOFE-VGA/TOFE/VGAIN_SCL: track 102.4 -> 37.9 mm, vias 2 -> 1
- net /TOFE-VGA/VGA/VGAOUT_HSYNC: track 4.69 -> 65.7 mm
- net /TOFE-VGA/AD9984/SOGOUT: track 0.00 -> 50.3 mm, vias 0 -> 1
- net /TOFE-VGA/AD9984/DATACK: track 0.00 -> 48.7 mm, vias 0 -> 1
- net /TOFE-VGA/VGA/VGAIN5V_SCL: track 45.7 -> 0.00 mm
- net /TOFE-VGA/VGA/VGAIN5V_SDA: track 41.4 -> 0.00 mm
- net /TOFE-VGA/AD9984/HSOUT: track 0.00 -> 40.4 mm, vias 0 -> 1
- net /HSOUT: track 38.0 -> 0.00 mm, vias 1 -> 0
- net /SOGOUT: track 37.4 -> 0.00 mm
- net /TOFE-VGA/VGA/VGAOUT_VSYNC: track 24.3 -> 59.8 mm
- net (no net): track 92.0 -> 56.7 mm, vias 13 -> 5
- net /DATACK: track 35.3 -> 0.00 mm, vias 1 -> 0
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Other:
- board size 46 x 3 mm -> 99 x 99 mm
- board text added: "& MANUFACTURER'S CODE ON BOTTOM"
- board text added: "+3.3V"
- board text added: "1 OZ CU ALL LAYERS, WHEN FINISHED"
- board text added: "1. MATERIAL: FR-4, 1.6mm THK, 4 LAYER"
- board text added: "1.75"
- board text added: "1.88"
- board text added: "11.0"
- board text added: "11.25"
- board text added: "12.5"
- board text added: "15.0"
- board text added: "18.25"
- board text added: "2. SOLDERMASK OVER BARE CU. HASL. RoHS"
- board text added: "2.5R"
- board text added: "2.75"
- board text added: "3. SILKSCREEN TOP AND BOTTOM, WHITE"
- board text added: "3.75"
- board text added: "3.75 REF"
- board text added: "38.25"
- board text added: "4. PERMANENTLY MARK DATE CODE"
- board text added: "4.75"
- board text added: "7.45"
- board text added: "8"
- board text added: "8.00"
- board text added: "8.25"
- board text added: "85.50"
- board text added: "9.00"
- board text added: "94.50"
- board text added: "99 X 99"
- board text added: "99.00"
- board text added: "99.00 REF"
- board text added: "ADD DIMENSIONS FOR P601 CUTOUTS"
- board text added: "ADD HOLE CHART"
- board text added: "DETAIL A"
- board text added: "IN"
- board text added: "NO SCALE"
- board text added: "NOTES: (UNLESS OTHERWISE SPECIFIED)"
- board text added: "NU"
- board text added: "OUT"
- board text added: "PLATED HOLES TO HAVE .022mm CU MIN"
- board text added: "PVD"
- board text added: "SEE DETAIL A"
- board text added: "TOP/FRONT"
- board text added: "VD"
